File: DualLM317BenchSupply/DualLM317BenchSupply.sch (KiCad schematic (older format))
At the start: 20 parts

Commit message: updating design to use 6 position switch to select current limiting resistor.
Parts:
- removed R?: 100, ~, symbol R
- removed R?: 10, ~, symbol R
- removed SW?: SWITCH_INV, ~, symbol SWITCH_INV
- added C?: 0.1uF, ~, symbol C
Connections:
- wire segments 43 -> 41
Other:
- note added: "Current Limiting"
- note added: "Status LED"
- note added: "Voltage Limiting"
- note removed: "10R = 125mA\n100R = 12.5mA"
- moved on the sheet: C?, D?, P?, RV?, U?

Commit message: adding input / output switches, revising schematic parts.
Parts:
- removed R?: 1k, ~, symbol R
- removed R?: 680, ~, symbol R
- removed SW?: SWITCH_INV, ~, symbol SWITCH_INV
- added R?: 680, ~, symbol R_0W25_1PCT
- added R?: 1k, ~, symbol R_0W25
- added SW? (x3): SPDT, ~, symbol SPDT
Connections:
- wire segments 41 -> 68
- no-connect marks 0 -> 3
Other:
- note added: "680 & 10k = 19.6V max"
- note added: "Output Enable / Disable"
- note added: "Power On / Off"
- note added: "Vin (24V DC)"
- note added: "Vout\n(1.25V - 19.6V DC)"
- note removed: "10k = 19.6V"
- note removed: "Vin (24V)"
- note removed: "Vout (1.25V - 19.6V)"
- moved on the sheet: C?, D?, P?, RV?, U?

Commit message: adding voltmeter and ammeter
Parts:
- added R?: 10M, ~, symbol R
- added R?: 0.05, ~, symbol R
Connections:
- wire segments 68 -> 72
Other:
- note added: "Ammeter"
- note added: "Voltmeter"
- moved on the sheet: C?, D?, P?, R?, RV?, SW?, U?

Commit message: annotating parts.  adding printout of schematic.
Parts:
- gave numbers to parts that had none: 22
Changed lines of the file:
@@
 $EndDescr
 $Comp
-L LM317 U?
+L LM317 U101
 U 1 1 53115585
 P 3600 3850
-F 0 "U?" H 3600 4150 60  0000 C CNN
+F 0 "U101" H 3600 4150 60  0000 C CNN
 F 1 "LM317" H 3650 3600 60  0000 L CNN
 F 2 "~" H 3600 3850 60  0000 C CNN
@@
 $EndComp
 $Comp
-L LM317 U?
+L LM317 U102
 U 1 1 53115594
 P 7300 3850
-F 0 "U?" H 7300 4150 60  0000 C CNN
+F 0 "U102" H 7300 4150 60  0000 C CNN
 F 1 "LM317" H 7350 3600 60  0000 L CNN
 F 2 "~" H 7300 3850 60  0000 C CNN
@@
 $EndComp
 $Comp
-L LED D?
+L LED D101
 U 1 1 531156EE
 P 2750 5800
-F 0 "D?" H 2750 5900 50  0000 C CNN
+F 0 "D101" H 2750 5900 50  0000 C CNN
 F 1 "LED" H 2750 5700 50  0000 C CNN
 F 2 "~" H 2750 5800 60  0000 C CNN
@@
 $EndComp
 $Comp
-L GND #PWR?
+L GND #PWR103
 U 1 1 5311570D
 P 2750 6700
-F 0 "#PWR?" H 2750 6700 30  0001 C CNN
+F 0 "#PWR103" H 2750 6700 30  0001 C CNN
 F 1 "GND" H 2750 6630 30  0001 C CNN
 F 2 "" H 2750 6700 60  0000 C CNN
@@
 $EndComp
 $Comp
-L CP1 C?
+L CP1 C102
 U 1 1 5311573B
 P 3000 4000
-F 0 "C?" H 3050 4100 50  0000 L CNN
+F 0 "C102" H 3050 4100 50  0000 L CNN
 F 1 "100uF" H 3050 3900 50  0000 L CNN
 F 2 "~" H 3000 4000 60  0000 C CNN
@@
 $EndComp
 $Comp
-L CP1 C?
+L CP1 C103
 U 1 1 5311574A
 P 6650 4000
-F 0 "C?" H 6700 4100 50  0000 L CNN
+F 0 "C103" H 6700 4100 50  0000 L CNN
 F 1 "1uF" H 6700 3900 50  0000 L CNN
 F 2 "~" H 6650 4000 60  0000 C CNN
@@
 $EndComp
 $Comp
-L GND #PWR?
+L GND #PWR105
 U 1 1 5311577C
 P 6650 4300
-F 0 "#PWR?" H 6650 4300 30  0001 C CNN
+F 0 "#PWR105" H 6650 4300 30  0001 C CNN
 F 1 "GND" H 6650 4230 30  0001 C CNN
 F 2 "" H 6650 4300 60  0000 C CNN
@@
 $EndComp
 $Comp
-L GND #PWR?
+L GND #PWR104
 U 1 1 531157E6
 P 3000 4300
-F 0 "#PWR?" H 3000 4300 30  0001 C CNN
+F 0 "#PWR104" H 3000 4300 30  0001 C CNN
 F 1 "GND" H 3000 4230 30  0001 C CNN
 F 2 "" H 3000 4300 60  0000 C CNN
@@
 $EndComp
 $Comp
-L POT RV?
+L POT RV101
 U 1 1 531160F8
 P 7850 4650
-F 0 "RV?" H 7850 4550 50  0000 C CNN
+F 0 "RV101" H 7850 4550 50  0000 C CNN
 F 1 "10k" H 7850 4650 50  0000 C CNN
 F 2 "~" H 7850 4650 60  0000 C CNN
@@
 $EndComp
 $Comp
-L GND #PWR?
+L GND #PWR107
 U 1 1 53116107
 P 7850 5000
-F 0 "#PWR?" H 7850 5000 30  0001 C CNN
+F 0 "#PWR107" H 7850 5000 30  0001 C CNN
 F 1 "GND" H 7850 4930 30  0001 C CNN
 F 2 "" H 7850 5000 60  0000 C CNN
@@
 $EndComp
 $Comp
-L CP1 C?
+L CP1 C104
 U 1 1 53116116
 P 7300 4700
-F 0 "C?" H 7350 4800 50  0000 L CNN
+F 0 "C104" H 7350 4800 50  0000 L CNN
 F 1 "10uF" H 7350 4600 50  0000 L CNN
 F 2 "~" H 7300 4700 60  0000 C CNN
@@
 $EndComp
 $Comp
-L GND #PWR?
+L GND #PWR106
 U 1 1 53116125
 P 7300 5000
-F 0 "#PWR?" H 7300 5000 30  0001 C CNN
+F 0 "#PWR106" H 7300 5000 30  0001 C CNN
 F 1 "GND" H 7300 4930 30  0001 C CNN
 F 2 "" H 7300 5000 60  0000 C CNN
@@
 $EndComp
 $Comp
-L DIODE D?
+L DIODE D103
 U 1 1 53116214
 P 8250 4000
-F 0 "D?" H 8250 4100 40  0000 C CNN
+F 0 "D103" H 8250 4100 40  0000 C CNN
 F 1 "1N4148" H 8250 3900 40  0000 C CNN
 F 2 "~" H 8250 4000 60  0000 C CNN
@@
 $EndComp
 $Comp
-L DIODE D?
+L DIODE D102
 U 1 1 53116272
 P 4950 1250
-F 0 "D?" H 4950 1350 40  0000 C CNN
+F 0 "D102" H 4950 1350 40  0000 C CNN
 F 1 "1N4148" H 4950 1150 40  0000 C CNN
 F 2 "~" H 4950 1250 60  0000 C CNN
@@
 Connection ~ 8350 3700
 $Comp
-L CP1 C?
+L CP1 C105
 U 1 1 5311632D
 P 8600 4000
-F 0 "C?" H 8650 4100 50  0000 L CNN
+F 0 "C105" H 8650 4100 50  0000 L CNN
 F 1 "1uF" H 8650 3900 50  0000 L CNN
 F 2 "~" H 8600 4000 60  0000 C CNN
@@
 Connection ~ 8600 3700
 $Comp
-L GND #PWR?
+L GND #PWR108
 U 1 1 531163B7
 P 8600 4300
-F 0 "#PWR?" H 8600 4300 30  0001 C CNN
+F 0 "#PWR108" H 8600 4300 30  0001 C CNN
 F 1 "GND" H 8600 4230 30  0001 C CNN
 F 2 "" H 8600 4300 60  0000 C CNN
@@
 Current Limit Bypass
 $Comp
-L CONN_1 P?
+L CONN_1 P103
 U 1 1 5311679A
 P 10500 3700
-F 0 "P?" H 10580 3700 40  0000 L CNN
+F 0 "P103" H 10580 3700 40  0000 L CNN
 F 1 "CONN_1" H 10500 3755 30  0001 C CNN
 F 2 "" H 10500 3700 60  0000 C CNN
@@
 $EndComp
 $Comp
-L CONN_1 P?
+L CONN_1 P104
 U 1 1 531167A9
 P 10500 4100
-F 0 "P?" H 10580 4100 40  0000 L CNN
+F 0 "P104" H 10580 4100 40  0000 L CNN
 F 1 "CONN_1" H 10500 4155 30  0001 C CNN
 F 2 "" H 10500 4100 60  0000 C CNN
@@
 $EndComp
 $Comp
-L GND #PWR?
+L GND #PWR110
 U 1 1 53116825
 P 10250 4200
-F 0 "#PWR?" H 10250 4200 30  0001 C CNN
+F 0 "#PWR110" H 10250 4200 30  0001 C CNN
 F 1 "GND" H 10250 4130 30  0001 C CNN
 F 2 "" H 10250 4200 60  0000 C CNN
@@
 Vout\n(1.25V - 19.6V DC)
 $Comp
-L CONN_1 P?
+L CONN_1 P101
 U 1 1 5311686A
 P 850 3700
-F 0 "P?" H 930 3700 40  0000 L CNN
+F 0 "P101" H 930 3700 40  0000 L CNN
 F 1 "CONN_1" H 850 3755 30  0001 C CNN
 F 2 "" H 850 3700 60  0000 C CNN
@@
 $EndComp
 $Comp
-L CONN_1 P?
+L CONN_1 P102
 U 1 1 53116879
 P 850 4050
-F 0 "P?" H 930 4050 40  0000 L CNN
+F 0 "P102" H 930 4050 40  0000 L CNN
 F 1 "CONN_1" H 850 4105 30  0001 C CNN
 F 2 "" H 850 4050 60  0000 C CNN
@@
 $EndComp
 $Comp
-L GND #PWR?
+L GND #PWR101
 U 1 1 53116888
 P 1100 4150
-F 0 "#PWR?" H 1100 4150 30  0001 C CNN
+F 0 "#PWR101" H 1100 4150 30  0001 C CNN
 F 1 "GND" H 1100 4080 30  0001 C CNN
 F 2 "" H 1100 4150 60  0000 C CNN
@@
 Connection ~ 5250 3700
 $Comp
-L C C?
+L C C101
 U 1 1 53255526
 P 2650 4000
-F 0 "C?" H 2650 4100 40  0000 L CNN
+F 0 "C101" H 2650 4100 40  0000 L CNN
 F 1 "0.1uF" H 2656 3915 40  0000 L CNN
 F 2 "~" H 2688 3850 30  0000 C CNN
@@
 $EndComp
 $Comp
-L GND #PWR?
+L GND #PWR102
 U 1 1 53255562
 P 2650 4300
-F 0 "#PWR?" H 2650 4300 30  0001 C CNN
+F 0 "#PWR102" H 2650 4300 30  0001 C CNN
 F 1 "GND" H 2650 4230 30  0001 C CNN
 F 2 "" H 2650 4300 60  0000 C CNN
@@
 	9100 3700 9250 3700
 $Comp
-L SPDT SW?
+L SPDT SW102
 U 1 1 5325CCF9
 P 3650 3000
-F 0 "SW?" H 3870 3100 40  0000 C CNN
+F 0 "SW102" H 3870 3100 40  0000 C CNN
 F 1 "SPDT" H 3930 2930 40  0000 C CNN
 F 2 "~" H 4030 3000 60  0000 C CNN
@@
 $EndComp
 $Comp
-L R_0W25_1PCT R?
+L R_0W25_1PCT R103
 U 1 1 5325DB3F
 P 7850 4050
-F 0 "R?" V 7930 4050 40  0000 C CNN
+F 0 "R103" V 7930 4050 40  0000 C CNN
 F 1 "680" V 7857 4051 40  0000 C CNN
 F 2 "~" V 7780 4050 30  0000 C CNN
@@
 $EndComp
 $Comp
-L R_0W25 R?
+L R_0W25 R101
 U 1 1 5325E3AD
 P 2750 6350
-F 0 "R?" V 2830 6350 40  0000 C CNN
+F 0 "R101" V 2830 6350 40  0000 C CNN
 F 1 "1k" V 2757 6351 40  0000 C CNN
 F 2 "~" V 2680 6350 30  0000 C CNN
@@
 $EndComp
 $Comp
-L SPDT SW?
+L SPDT SW101
 U 1 1 5325E539
 P 1350 3700
-F 0 "SW?" H 1570 3800 40  0000 C CNN
+F 0 "SW101" H 1570 3800 40  0000 C CNN
 F 1 "SPDT" H 1630 3630 40  0000 C CNN
 F 2 "~" H 1730 3700 60  0000 C CNN
@@
 	8350 1250 5150 1250
 $Comp
-L SPDT SW?
+L SPDT SW103
 U 1 1 53260847
 P 9250 3700
-F 0 "SW?" H 9470 3800 40  0000 C CNN
+F 0 "SW103" H 9470 3800 40  0000 C CNN
 F 1 "SPDT" H 9530 3630 40  0000 C CNN
 F 2 "~" H 9630 3700 60  0000 C CNN
@@
 Output Enable / Disable
 $Comp
-L R R?
+L R R104
 U 1 1 5325DA41
 P 9700 2100
-F 0 "R?" V 9780 2100 40  0000 C CNN
+F 0 "R104" V 9780 2100 40  0000 C CNN
 F 1 "10M" V 9707 2101 40  0000 C CNN
 F 2 "~" V 9630 2100 30  0000 C CNN
@@
 $EndComp
 $Comp
-L GND #PWR?
+L GND #PWR109
 U 1 1 5325DAA8
 P 10050 2200
-F 0 "#PWR?" H 10050 2200 30  0001 C CNN
+F 0 "#PWR109" H 10050 2200 30  0001 C CNN
 F 1 "GND" H 10050 2130 30  0001 C CNN
 F 2 "" H 10050 2200 60  0000 C CNN
@@
 Voltmeter
 $Comp
-L R R?
+L R R102
 U 1 1 5325DFC4
 P 5950 3700
-F 0 "R?" V 6030 3700 40  0000 C CNN
+F 0 "R102" V 6030 3700 40  0000 C CNN
 F 1 "0.05" V 5957 3701 40  0000 C CNN
 F 2 "~" V 5880 3700 30  0000 C CNN

Commit message: adding voltmeter / ammeter
Parts:
- removed R102: 0.05, ~, symbol R
- removed R104: 10M, ~, symbol R
- added C?: 10uF, ~, symbol CP1
- added C?: 0.1uF, ~, symbol C
- added DS?: AMMETER, ~, symbol AMMETER
- added DS?: VOLTMETER, ~, symbol VOLTMETER
- added U?: 7805, ~, symbol 7805
- C102: value 100uF -> 1000uF
- R103: value 680 -> 330
- RV101: value 10k -> 5k
Connections:
- net labels added: 5V
- wire segments 72 -> 69
Other:
- note added: "330 & 5k = 20.2V max\n330 = 3.8mA error"
- note added: "5V Supply"
- note added: "Vout\n(1.25V - 20.2V DC)"
- note removed: "680 & 10k = 19.6V max"
- note removed: "Ammeter"
- note removed: "Voltmeter"
- note removed: "Vout\n(1.25V - 19.6V DC)"
- moved on the sheet: C101, C102, C103, C104, C105, D101, D102, D103, P101, P102, P103, P104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

Commit message: revising protection diodes
Parts:
- removed P101, P102: CONN_1, symbol CONN_1
- added CON101: BARREL_JACK, symbol BARREL_JACK
- added D104: 1N4148, ~, symbol DIODE
- gave numbers to parts that had none: 5
Connections:
- wire segments 69 -> 74
Other:
- moved on the sheet: C101, C102, C103, C104, C105, C106, C107, D101, D102, D103, P103, P104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

Commit message: updating switch
Parts:
- CON101: footprint (none) -> ~
Changed lines of the file:
@@
 EESchema Schematic File Version 2
+LIBS:connectors_PL
 LIBS:displays_PL
 LIBS:resistors_PL
@@
 	5800 6300 5800 4200
 Connection ~ 5800 4200
-$Comp
-L BARREL_JACK CON101
-U 1 1 53267050
-P 2200 4300
-F 0 "CON101" H 2200 4550 60  0000 C CNN
-F 1 "BARREL_JACK" H 2200 4100 60  0000 C CNN
-F 2 "" H 2200 4300 60  0000 C CNN
-F 3 "" H 2200 4300 60  0000 C CNN
-	1    2200 4300
-	1    0    0    -1
-$EndComp
 Wire Wire Line
 	2500 4300 2600 4300
@@
 Wire Wire Line
 	3150 4200 2500 4200
+$Comp
+L BARREL_JACK CON101
+U 1 1 53265EFE
+P 2200 4300
+F 0 "CON101" H 2200 4500 40  0000 C CNN
+F 1 "BARREL_JACK" H 2200 4150 40  0000 C CNN
+F 2 "~" H 2200 4300 60  0000 C CNN
+F 3 "~" H 2200 4300 60  0000 C CNN
+	1    2200 4300
+	1    0    0    -1
+$EndComp
 $EndSCHEMATC
