File: DualLM317BenchSupply/DualLM317BenchSupply.sch (KiCad schematic (older format))
At the start: 25 parts, among them CON101 BARREL_JACK, P103 CONN_1, P104 CONN_1, SW101 SPDT, SW102 SPDT, SW103 SPDT, U101 LM317, U102 LM317, U103 7805

Commit message: updating parts
Parts:
- removed C101, C106: 0.1uF, ~, symbol C
- removed C102: 1000uF, ~, symbol CP1
- removed C103, C105: 1uF, ~, symbol CP1
- removed C104, C107: 10uF, ~, symbol CP1
- removed U101, U102: LM317, ~, symbol LM317
- removed U103: 7805, ~, symbol 7805
- added C101, C106: 0.1uF, ~, symbol C_CER
- added C102: 1000uF, ~, symbol C_EL
- added C103, C105: 1uF, ~, symbol C_EL
- added C104, C107: 10uF, ~, symbol C_EL
- added U?: 7805, ~, symbol 7805
- added U? (x2): LM317, ~, symbol LM317
Changed lines of the file:
@@
 EESchema Schematic File Version 2
+LIBS:regulators_PL
+LIBS:capacitors_PL
 LIBS:connectors_PL
 LIBS:displays_PL
@@
 $EndDescr
 $Comp
-L LM317 U101
-U 1 1 53115585
-P 7150 4350
-F 0 "U101" H 7150 4650 60  0000 C CNN
-F 1 "LM317" H 7200 4100 60  0000 L CNN
-F 2 "~" H 7150 4350 60  0000 C CNN
-F 3 "~" H 7150 4350 60  0000 C CNN
-	1    7150 4350
-	1    0    0    -1
-$EndComp
-$Comp
-L LM317 U102
-U 1 1 53115594
-P 11500 4350
-F 0 "U102" H 11500 4650 60  0000 C CNN
-F 1 "LM317" H 11550 4100 60  0000 L CNN
-F 2 "~" H 11500 4350 60  0000 C CNN
-F 3 "~" H 11500 4350 60  0000 C CNN
-	1    11500 4350
-	1    0    0    -1
-$EndComp
-$Comp
 L LED D101
 U 1 1 531156EE
@@
 $EndComp
 $Comp
-L GND #PWR01
+L GND #PWR103
 U 1 1 5311570D
 P 5200 6000
-F 0 "#PWR01" H 5200 6000 30  0001 C CNN
+F 0 "#PWR103" H 5200 6000 30  0001 C CNN
 F 1 "GND" H 5200 5930 30  0001 C CNN
 F 2 "" H 5200 6000 60  0000 C CNN
@@
 $EndComp
 $Comp
-L CP1 C102
-U 1 1 5311573B
-P 4300 4500
-F 0 "C102" H 4350 4600 50  0000 L CNN
-F 1 "1000uF" H 4350 4400 50  0000 L CNN
-F 2 "~" H 4300 4500 60  0000 C CNN
-F 3 "~" H 4300 4500 60  0000 C CNN
-	1    4300 4500
-	1    0    0    -1
-$EndComp
-$Comp
-L CP1 C103
-U 1 1 5311574A
-P 10850 4500
-F 0 "C103" H 10900 4600 50  0000 L CNN
-F 1 "1uF" H 10900 4400 50  0000 L CNN
-F 2 "~" H 10850 4500 60  0000 C CNN
-F 3 "~" H 10850 4500 60  0000 C CNN
-	1    10850 4500
-	1    0    0    -1
-$EndComp
-$Comp
-L GND #PWR02
+L GND #PWR109
 U 1 1 5311577C
 P 10850 4800
-F 0 "#PWR02" H 10850 4800 30  0001 C CNN
+F 0 "#PWR109" H 10850 4800 30  0001 C CNN
 F 1 "GND" H 10850 4730 30  0001 C CNN
 F 2 "" H 10850 4800 60  0000 C CNN
@@
 $EndComp
 $Comp
-L GND #PWR03
+L GND #PWR102
 U 1 1 531157E6
 P 4300 4800
-F 0 "#PWR03" H 4300 4800 30  0001 C CNN
+F 0 "#PWR102" H 4300 4800 30  0001 C CNN
 F 1 "GND" H 4300 4730 30  0001 C CNN
 F 2 "" H 4300 4800 60  0000 C CNN
@@
 $EndComp
 $Comp
-L GND #PWR04
+L GND #PWR111
 U 1 1 53116107
 P 12050 5500
-F 0 "#PWR04" H 12050 5500 30  0001 C CNN
+F 0 "#PWR111" H 12050 5500 30  0001 C CNN
 F 1 "GND" H 12050 5430 30  0001 C CNN
 F 2 "" H 12050 5500 60  0000 C CNN
@@
 $EndComp
 $Comp
-L CP1 C104
-U 1 1 53116116
-P 11500 5200
-F 0 "C104" H 11550 5300 50  0000 L CNN
-F 1 "10uF" H 11550 5100 50  0000 L CNN
-F 2 "~" H 11500 5200 60  0000 C CNN
-F 3 "~" H 11500 5200 60  0000 C CNN
-	1    11500 5200
-	1    0    0    -1
-$EndComp
-$Comp
-L GND #PWR05
+L GND #PWR110
 U 1 1 53116125
 P 11500 5500
-F 0 "#PWR05" H 11500 5500 30  0001 C CNN
+F 0 "#PWR110" H 11500 5500 30  0001 C CNN
 F 1 "GND" H 11500 5430 30  0001 C CNN
 F 2 "" H 11500 5500 60  0000 C CNN
@@
 $EndComp
 Wire Wire Line
-	8800 5000 7150 5000
-Wire Wire Line
-	7150 5000 7150 4700
+	7150 5000 8800 5000
+Wire Wire Line
+	7150 4500 7150 5000
 Wire Wire Line
 	5200 5900 5200 6000
@@
 	4300 4700 4300 4800
 Wire Wire Line
-	11500 4700 11500 5000
+	11500 4500 11500 5000
 Wire Wire Line
 	11500 5400 11500 5500
@@
 Connection ~ 12450 4200
 Connection ~ 12000 4200
-$Comp
-L CP1 C105
-U 1 1 5311632D
-P 12800 4500
-F 0 "C105" H 12850 4600 50  0000 L CNN
-F 1 "1uF" H 12850 4400 50  0000 L CNN
-F 2 "~" H 12800 4500 60  0000 C CNN
-F 3 "~" H 12800 4500 60  0000 C CNN
-	1    12800 4500
-	1    0    0    -1
-$EndComp
 Wire Wire Line
 	12800 4200 12800 4300
 Connection ~ 12800 4200
 $Comp
-L GND #PWR06
+L GND #PWR112
 U 1 1 531163B7
 P 12800 4800
-F 0 "#PWR06" H 12800 4800 30  0001 C CNN
+F 0 "#PWR112" H 12800 4800 30  0001 C CNN
 F 1 "GND" H 12800 4730 30  0001 C CNN
 F 2 "" H 12800 4800 60  0000 C CNN
@@
 $EndComp
 $Comp
-L GND #PWR07
+L GND #PWR114
 U 1 1 53116825
 P 14600 4700
-F 0 "#PWR07" H 14600 4700 30  0001 C CNN
+F 0 "#PWR114" H 14600 4700 30  0001 C CNN
 F 1 "GND" H 14600 4630 30  0001 C CNN
 F 2 "" H 14600 4700 60  0000 C CNN
@@
 Vout\n(1.25V - 20.2V DC)
 $Comp
-L GND #PWR08
+L GND #PWR101
 U 1 1 53116888
 P 2600 4500
-F 0 "#PWR08" H 2600 4500 30  0001 C CNN
+F 0 "#PWR101" H 2600 4500 30  0001 C CNN
 F 1 "GND" H 2600 4430 30  0001 C CNN
 F 2 "" H 2600 4500 60  0000 C CNN
@@
 $EndSheet
 Wire Wire Line
-	7550 4200 7800 4200
+	7450 4200 7800 4200
 Connection ~ 7650 4200
 Wire Wire Line
@@
 Connection ~ 8800 4200
 $Comp
-L C C101
-U 1 1 53255526
-P 6300 4500
-F 0 "C101" H 6300 4600 40  0000 L CNN
-F 1 "0.1uF" H 6306 4415 40  0000 L CNN
-F 2 "~" H 6338 4350 30  0000 C CNN
-F 3 "~" H 6300 4500 60  0000 C CNN
-	1    6300 4500
-	1    0    0    -1
-$EndComp
-$Comp
-L GND #PWR09
+L GND #PWR105
 U 1 1 53255562
 P 6300 4800
-F 0 "#PWR09" H 6300 4800 30  0001 C CNN
+F 0 "#PWR105" H 6300 4800 30  0001 C CNN
 F 1 "GND" H 6300 4730 30  0001 C CNN
 F 2 "" H 6300 4800 60  0000 C CNN
@@
 	8650 4200 9850 4200
 Wire Wire Line
-	10350 4200 11100 4200
+	10350 4200 11200 4200
 Wire Notes Line
 	6050 2800 9050 2800
@@
 	13150 5750 13150 3400
 Wire Wire Line
-	11900 4200 13600 4200
+	11800 4200 13600 4200
 $Comp
 L SPDT SW102
@@
 	3950 4100 3950 4200
 Wire Wire Line
-	3950 4200 6750 4200
+	3950 4200 6850 4200
 Text Notes 3300 4000 0    40   ~ 0
 Power On / Off
@@
 330 & 5k = 20.2V max\n330 = 3.8mA error
 $Comp
-L 7805 U103
-U 1 1 532639FA
-P 6750 6350
-F 0 "U103" H 6900 6154 60  0000 C CNN
-F 1 "7805" H 6750 6550 60  0000 C CNN
-F 2 "~" H 6750 6350 60  0000 C CNN
-F 3 "~" H 6750 6350 60  0000 C CNN
-	1    6750 6350
-	1    0    0    -1
-$EndComp
-$Comp
-L GND #PWR010
+L GND #PWR106
 U 1 1 53264209
 P 6750 6700
-F 0 "#PWR010" H 6750 6700 30  0001 C CNN
+F 0 "#PWR106" H 6750 6700 30  0001 C CNN
 F 1 "GND" H 6750 6630 30  0001 C CNN
 F 2 "" H 6750 6700 60  0000 C CNN
@@
 $EndComp
 $Comp
-L CP1 C107
-U 1 1 5326428D
-P 7250 6600
-F 0 "C107" H 7300 6700 50  0000 L CNN
-F 1 "10uF" H 7300 6500 50  0000 L CNN
-F 2 "~" H 7250 6600 60  0000 C CNN
-F 3 "~" H 7250 6600 60  0000 C CNN
-	1    7250 6600
-	1    0    0    -1
-$EndComp
-$Comp
-L GND #PWR011
+L GND #PWR107
 U 1 1 532642AB
 P 7250 6900
-F 0 "#PWR011" H 7250 6900 30  0001 C CNN
+F 0 "#PWR107" H 7250 6900 30  0001 C CNN
 F 1 "GND" H 7250 6830 30  0001 C CNN
 F 2 "" H 7250 6900 60  0000 C CNN
@@
 	7250 6400 7250 6300
 Wire Wire Line
-	7150 6300 7350 6300
+	7050 6300 7350 6300
 Wire Wire Line
 	7350 6300 7350 6200
@@
 5V
 Wire Wire Line
-	5800 6300 6350 6300
-$Comp
-L C C106
-U 1 1 53264954
-P 6250 6600
-F 0 "C106" H 6250 6700 40  0000 L CNN
-F 1 "0.1uF" H 6256 6515 40  0000 L CNN
-F 2 "~" H 6288 6450 30  0000 C CNN
-F 3 "~" H 6250 6600 60  0000 C CNN
-	1    6250 6600
-	1    0    0    -1
-$EndComp
-$Comp
-L GND #PWR012
+	5800 6300 6450 6300
+$Comp
+L GND #PWR104
 U 1 1 5326496C
 P 6250 6900
-F 0 "#PWR012" H 6250 6900 30  0001 C CNN
+F 0 "#PWR104" H 6250 6900 30  0001 C CNN
 F 1 "GND" H 6250 6830 30  0001 C CNN
 F 2 "" H 6250 6900 60  0000 C CNN
@@
 $EndComp
 $Comp
-L GND #PWR013
+L GND #PWR113
 U 1 1 5326745C
 P 13500 3200
-F 0 "#PWR013" H 13500 3200 30  0001 C CNN
+F 0 "#PWR113" H 13500 3200 30  0001 C CNN
 F 1 "GND" H 13500 3130 30  0001 C CNN
 F 2 "" H 13500 3200 60  0000 C CNN
@@
 5V
 $Comp
-L GND #PWR014
+L GND #PWR108
 U 1 1 53267BC5
 P 9350 4100
-F 0 "#PWR014" H 9350 4100 30  0001 C CNN
+F 0 "#PWR108" H 9350 4100 30  0001 C CNN
 F 1 "GND" H 9350 4030 30  0001 C CNN
 F 2 "" H 9350 4100 60  0000 C CNN
@@
 	1    0    0    -1
 $EndComp
+$Comp
+L C_CER C106
+U 1 1 53268218
+P 6250 6600
+F 0 "C106" H 6270 6660 30  0000 L BNN
+F 1 "0.1uF" H 6270 6540 30  0000 L TNN
+F 2 "~" H 6288 6450 30  0000 C CNN
+F 3 "~" H 6250 6600 60  0000 C CNN
+	1    6250 6600
+	1    0    0    -1
+$EndComp
+$Comp
+L C_EL C107
+U 1 1 53268227
+P 7250 6600
+F 0 "C107" H 7270 6660 30  0000 L BNN
+F 1 "10uF" H 7270 6510 30  0000 L TNN
+F 2 "~" H 7288 6450 30  0000 C CNN
+F 3 "~" H 7250 6600 60  0000 C CNN
+	1    7250 6600
+	1    0    0    -1
+$EndComp
+$Comp
+L C_EL C102
+U 1 1 53268786
+P 4300 4500
+F 0 "C102" H 4320 4560 30  0000 L BNN
+F 1 "1000uF" H 4320 4410 30  0000 L TNN
+F 2 "~" H 4338 4350 30  0000 C CNN
+F 3 "~" H 4300 4500 60  0000 C CNN
+	1    4300 4500
+	1    0    0    -1
+$EndComp
+$Comp
+L C_CER C101
+U 1 1 53268930
+P 6300 4500
+F 0 "C101" H 6320 4560 30  0000 L BNN
+F 1 "0.1uF" H 6320 4440 30  0000 L TNN
+F 2 "~" H 6338 4350 30  0000 C CNN
+F 3 "~" H 6300 4500 60  0000 C CNN
+	1    6300 4500
+	1    0    0    -1
+$EndComp
+$Comp
+L C_EL C103
+U 1 1 53268CD2
+P 10850 4500
+F 0 "C103" H 10870 4560 30  0000 L BNN
+F 1 "1uF" H 10870 4410 30  0000 L TNN
+F 2 "~" H 10888 4350 30  0000 C CNN
+F 3 "~" H 10850 4500 60  0000 C CNN
+	1    10850 4500
+	1    0    0    -1
+$EndComp
+$Comp
+L C_EL C104
+U 1 1 53268E70
+P 11500 5200
+F 0 "C104" H 11520 5260 30  0000 L BNN
+F 1 "10uF" H 11520 5110 30  0000 L TNN
+F 2 "~" H 11538 5050 30  0000 C CNN
+F 3 "~" H 11500 5200 60  0000 C CNN
+	1    11500 5200
+	1    0    0    -1
+$EndComp
+$Comp
+L C_EL C105
+U 1 1 53269020
+P 12800 4500
+F 0 "C105" H 12820 4560 30  0000 L BNN
+F 1 "1uF" H 12820 4410 30  0000 L TNN
+F 2 "~" H 12838 4350 30  0000 C CNN
+F 3 "~" H 12800 4500 60  0000 C CNN
+	1    12800 4500
+	1    0    0    -1
+$EndComp
+$Comp
+L 7805 U?
+U 1 1 5326A1C4
+P 6750 6350
+F 0 "U?" H 6550 6510 40  0000 L BNN
+F 1 "7805" H 6950 6180 40  0000 R TNN
+F 2 "~" H 6750 6350 60  0000 C CNN
+F 3 "~" H 6750 6350 60  0000 C CNN
+	1    6750 6350
+	1    0    0    -1
+$EndComp
+$Comp
+L LM317 U?
+U 1 1 5326A2AB
+P 7150 4250
+F 0 "U?" H 6950 4410 40  0000 L BNN
+F 1 "LM317" H 7350 4080 40  0000 R TNN
+F 2 "~" H 7150 4250 60  0000 C CNN
+F 3 "~" H 7150 4250 60  0000 C CNN
+	1    7150 4250
+	1    0    0    -1
+$EndComp
+$Comp
+L LM317 U?
+U 1 1 5326A5B6
+P 11500 4250
+F 0 "U?" H 11300 4410 40  0000 L BNN
+F 1 "LM317" H 11700 4080 40  0000 R TNN
+F 2 "~" H 11500 4250 60  0000 C CNN
+F 3 "~" H 11500 4250 60  0000 C CNN
+	1    11500 4250
+	1    0    0    -1
+$EndComp

Commit message: updating switches, capacitors, and LEDs
Parts:
- gave numbers to parts that had none: 3
Changed lines of the file:
@@
 EESchema Schematic File Version 2
+LIBS:LEDs_PL
 LIBS:regulators_PL
 LIBS:capacitors_PL
@@
 $EndDescr
 $Comp
-L LED D101
-U 1 1 531156EE
-P 5200 5100
-F 0 "D101" H 5200 5200 50  0000 C CNN
-F 1 "LED" H 5200 5000 50  0000 C CNN
-F 2 "~" H 5200 5100 60  0000 C CNN
-F 3 "~" H 5200 5100 60  0000 C CNN
-	1    5200 5100
-	0    1    1    0
-$EndComp
-$Comp
 L GND #PWR103
 U 1 1 5311570D
@@
 	11800 4200 13600 4200
 $Comp
-L SPDT SW102
-U 1 1 5325CCF9
-P 7200 3500
-F 0 "SW102" H 7420 3600 40  0000 C CNN
-F 1 "SPDT" H 7480 3430 40  0000 C CNN
-F 2 "~" H 7580 3500 60  0000 C CNN
-F 3 "~" H 7580 3500 60  0000 C CNN
-	1    7200 3500
-	1    0    0    -1
-$EndComp
-$Comp
 L R_0W25_1PCT R103
 U 1 1 5325DB3F
@@
 	1    0    0    -1
 $EndComp
-$Comp
-L SPDT SW101
-U 1 1 5325E539
-P 3150 4200
-F 0 "SW101" H 3370 4300 40  0000 C CNN
-F 1 "SPDT" H 3430 4130 40  0000 C CNN
-F 2 "~" H 3530 4200 60  0000 C CNN
-F 3 "~" H 3530 4200 60  0000 C CNN
-	1    3150 4200
-	1    0    0    -1
-$EndComp
 Wire Wire Line
 	3800 4100 3950 4100
@@
 Text Notes 3300 4000 0    40   ~ 0
 Power On / Off
-$Comp
-L SPDT SW103
-U 1 1 53260847
-P 13600 4200
-F 0 "SW103" H 13820 4300 40  0000 C CNN
-F 1 "SPDT" H 13880 4130 40  0000 C CNN
-F 2 "~" H 13980 4200 60  0000 C CNN
-F 3 "~" H 13980 4200 60  0000 C CNN
-	1    13600 4200
-	1    0    0    -1
-$EndComp
 Wire Wire Line
 	14250 4100 14350 4100
@@
 $EndComp
 $Comp
-L 7805 U?
+L 7805 U101
 U 1 1 5326A1C4
 P 6750 6350
-F 0 "U?" H 6550 6510 40  0000 L BNN
+F 0 "U101" H 6550 6510 40  0000 L BNN
 F 1 "7805" H 6950 6180 40  0000 R TNN
 F 2 "~" H 6750 6350 60  0000 C CNN
@@
 $EndComp
 $Comp
-L LM317 U?
+L LM317 U102
 U 1 1 5326A2AB
 P 7150 4250
-F 0 "U?" H 6950 4410 40  0000 L BNN
+F 0 "U102" H 6950 4410 40  0000 L BNN
 F 1 "LM317" H 7350 4080 40  0000 R TNN
 F 2 "~" H 7150 4250 60  0000 C CNN
@@
 $EndComp
 $Comp
-L LM317 U?
+L LM317 U103
 U 1 1 5326A5B6
 P 11500 4250
-F 0 "U?" H 11300 4410 40  0000 L BNN
+F 0 "U103" H 11300 4410 40  0000 L BNN
 F 1 "LM317" H 11700 4080 40  0000 R TNN
 F 2 "~" H 11500 4250 60  0000 C CNN
@@
 	1    0    0    -1
 $EndComp
+$Comp
+L SPDT SW101
+U 1 1 5326AD65
+P 3150 4200
+F 0 "SW101" H 3370 4300 40  0000 C CNN
+F 1 "SPDT" H 3430 4130 40  0000 C CNN
+F 2 "~" H 3530 4200 60  0000 C CNN
+F 3 "~" H 3530 4200 60  0000 C CNN
+	1    3150 4200
+	1    0    0    -1
+$EndComp
+$Comp
+L SPDT SW102
+U 1 1 5326AE64
+P 7200 3500
+F 0 "SW102" H 7420 3600 40  0000 C CNN
+F 1 "SPDT" H 7480 3430 40  0000 C CNN
+F 2 "~" H 7580 3500 60  0000 C CNN
+F 3 "~" H 7580 3500 60  0000 C CNN
+	1    7200 3500
+	1    0    0    -1
+$EndComp
+$Comp
+L SPDT SW103
+U 1 1 5326AF75
+P 13600 4200
+F 0 "SW103" H 13820 4300 40  0000 C CNN
+F 1 "SPDT" H 13880 4130 40  0000 C CNN
+F 2 "~" H 13980 4200 60  0000 C CNN
+F 3 "~" H 13980 4200 60  0000 C CNN
+	1    13600 4200
+	1    0    0    -1
+$EndComp
+$Comp
+L LED D101
+U 1 1 5326B9A5
+P 5200 5100
+F 0 "D101" H 5075 5200 40  0000 C CNN
+F 1 "LED" H 5325 5200 30  0000 C CNN
+F 2 "~" H 5200 5100 60  0000 C CNN
+F 3 "~" H 5200 5100 60  0000 C CNN
+	1    5200 5100
+	0    1    1    0
+$EndComp
 $EndSCHEMATC
