File: DualLM317BenchSupply/DualLM317BenchSupply.sch (KiCad schematic (older format))
At the start: 25 parts, among them CON101 BARREL_JACK, P103 CONN_1, P104 CONN_1, SW101 SPDT, SW102 SPDT, SW103 SPDT, U101 7805, U102 LM317, U103 LM317

Commit message: reconfiguring protection diodes
Parts:
- added D1: 1N4148, ~, symbol DIODE
- C102: value 1000uF -> 100uF
Connections:
- wire segments 74 -> 80
Other:
- note added: "330 & 5k = 20.2V max\n330 = 3.8mA ammeter error"
- note removed: "330 & 5k = 20.2V max\n330 = 3.8mA error"
- moved on the sheet: C104, D102, D103, R103, RV101
Changed lines of the file:
@@
 Sheet 1 2
 Title ""
-Date "17 mar 2014"
+Date "18 mar 2014"
 Rev ""
 Comp ""
@@
 $EndDescr
 $Comp
-L GND #PWR103
+L GND #PWR3
 U 1 1 5311570D
 P 5200 6000
-F 0 "#PWR103" H 5200 6000 30  0001 C CNN
+F 0 "#PWR3" H 5200 6000 30  0001 C CNN
 F 1 "GND" H 5200 5930 30  0001 C CNN
 F 2 "" H 5200 6000 60  0000 C CNN
@@
 $EndComp
 $Comp
-L GND #PWR109
+L GND #PWR9
 U 1 1 5311577C
 P 10850 4800
-F 0 "#PWR109" H 10850 4800 30  0001 C CNN
+F 0 "#PWR9" H 10850 4800 30  0001 C CNN
 F 1 "GND" H 10850 4730 30  0001 C CNN
 F 2 "" H 10850 4800 60  0000 C CNN
@@
 $EndComp
 $Comp
-L GND #PWR102
+L GND #PWR2
 U 1 1 531157E6
 P 4300 4800
-F 0 "#PWR102" H 4300 4800 30  0001 C CNN
+F 0 "#PWR2" H 4300 4800 30  0001 C CNN
 F 1 "GND" H 4300 4730 30  0001 C CNN
 F 2 "" H 4300 4800 60  0000 C CNN
@@
 L POT RV101
 U 1 1 531160F8
-P 12050 5150
-F 0 "RV101" H 12050 5050 50  0000 C CNN
-F 1 "5k" H 12050 5150 50  0000 C CNN
-F 2 "~" H 12050 5150 60  0000 C CNN
-F 3 "~" H 12050 5150 60  0000 C CNN
-	1    12050 5150
+P 12200 5400
+F 0 "RV101" H 12200 5300 50  0000 C CNN
+F 1 "5k" H 12200 5400 50  0000 C CNN
+F 2 "~" H 12200 5400 60  0000 C CNN
+F 3 "~" H 12200 5400 60  0000 C CNN
+	1    12200 5400
 	0    -1   -1   0
 $EndComp
 $Comp
-L GND #PWR111
+L GND #PWR10
 U 1 1 53116107
-P 12050 5500
-F 0 "#PWR111" H 12050 5500 30  0001 C CNN
-F 1 "GND" H 12050 5430 30  0001 C CNN
-F 2 "" H 12050 5500 60  0000 C CNN
-F 3 "" H 12050 5500 60  0000 C CNN
-	1    12050 5500
-	1    0    0    -1
-$EndComp
-$Comp
-L GND #PWR110
+P 12200 5750
+F 0 "#PWR10" H 12200 5750 30  0001 C CNN
+F 1 "GND" H 12200 5680 30  0001 C CNN
+F 2 "" H 12200 5750 60  0000 C CNN
+F 3 "" H 12200 5750 60  0000 C CNN
+	1    12200 5750
+	1    0    0    -1
+$EndComp
+$Comp
+L GND #PWR11
 U 1 1 53116125
-P 11500 5500
-F 0 "#PWR110" H 11500 5500 30  0001 C CNN
-F 1 "GND" H 11500 5430 30  0001 C CNN
-F 2 "" H 11500 5500 60  0000 C CNN
-F 3 "" H 11500 5500 60  0000 C CNN
-	1    11500 5500
+P 12500 5750
+F 0 "#PWR11" H 12500 5750 30  0001 C CNN
+F 1 "GND" H 12500 5680 30  0001 C CNN
+F 2 "" H 12500 5750 60  0000 C CNN
+F 3 "" H 12500 5750 60  0000 C CNN
+	1    12500 5750
 	1    0    0    -1
 $EndComp
@@
 L DIODE D103
 U 1 1 53116214
-P 12450 4500
-F 0 "D103" H 12450 4600 40  0000 C CNN
-F 1 "1N4148" H 12450 4400 40  0000 C CNN
-F 2 "~" H 12450 4500 60  0000 C CNN
-F 3 "~" H 12450 4500 60  0000 C CNN
-	1    12450 4500
+P 11900 4500
+F 0 "D103" H 11900 4600 40  0000 C CNN
+F 1 "1N4148" H 11900 4400 40  0000 C CNN
+F 2 "~" H 11900 4500 60  0000 C CNN
+F 3 "~" H 11900 4500 60  0000 C CNN
+	1    11900 4500
 	0    -1   -1   0
 $EndComp
@@
 L DIODE D102
 U 1 1 53116272
-P 11500 3750
-F 0 "D102" H 11500 3850 40  0000 C CNN
-F 1 "1N4148" H 11500 3650 40  0000 C CNN
-F 2 "~" H 11500 3750 60  0000 C CNN
-F 3 "~" H 11500 3750 60  0000 C CNN
-	1    11500 3750
+P 11500 3850
+F 0 "D102" H 11500 3950 40  0000 C CNN
+F 1 "1N4148" H 11500 3750 40  0000 C CNN
+F 2 "~" H 11500 3850 60  0000 C CNN
+F 3 "~" H 11500 3850 60  0000 C CNN
+	1    11500 3850
 	-1   0    0    1
 $EndComp
@@
 	4300 4700 4300 4800
 Wire Wire Line
-	11500 4500 11500 5000
-Wire Wire Line
-	11500 5400 11500 5500
-Wire Wire Line
-	12050 5400 12050 5500
-Wire Wire Line
-	12050 4800 12050 4900
-Wire Wire Line
-	11500 4850 12450 4850
-Connection ~ 11500 4850
-Connection ~ 12050 4850
-Wire Wire Line
-	12050 4200 12050 4300
+	11500 4900 12200 4900
+Connection ~ 11900 4200
+Connection ~ 12200 4200
 Connection ~ 12050 4200
-Wire Wire Line
-	12450 4850 12450 4700
-Wire Wire Line
-	12450 4200 12450 4300
-Connection ~ 12450 4200
-Connection ~ 12000 4200
 Wire Wire Line
 	12800 4200 12800 4300
 Connection ~ 12800 4200
 $Comp
-L GND #PWR112
+L GND #PWR12
 U 1 1 531163B7
 P 12800 4800
-F 0 "#PWR112" H 12800 4800 30  0001 C CNN
+F 0 "#PWR12" H 12800 4800 30  0001 C CNN
 F 1 "GND" H 12800 4730 30  0001 C CNN
 F 2 "" H 12800 4800 60  0000 C CNN
@@
 Wire Wire Line
 	12800 4700 12800 4800
-Wire Wire Line
-	11900 5150 11850 5150
-Wire Wire Line
-	11850 5150 11850 5450
-Wire Wire Line
-	11850 5450 12050 5450
-Connection ~ 12050 5450
 Text Notes 7200 3300 0    40   ~ 0
 Current Limit Bypass
@@
 $EndComp
 $Comp
-L GND #PWR114
+L GND #PWR14
 U 1 1 53116825
 P 14600 4700
-F 0 "#PWR114" H 14600 4700 30  0001 C CNN
+F 0 "#PWR14" H 14600 4700 30  0001 C CNN
 F 1 "GND" H 14600 4630 30  0001 C CNN
 F 2 "" H 14600 4700 60  0000 C CNN
@@
 Vout\n(1.25V - 20.2V DC)
 $Comp
-L GND #PWR101
+L GND #PWR1
 U 1 1 53116888
 P 2600 4500
-F 0 "#PWR101" H 2600 4500 30  0001 C CNN
+F 0 "#PWR1" H 2600 4500 30  0001 C CNN
 F 1 "GND" H 2600 4430 30  0001 C CNN
 F 2 "" H 2600 4500 60  0000 C CNN
@@
 Text Notes 1850 3950 0    60   ~ 0
 Vin (24V DC)
-Connection ~ 6450 4200
+Connection ~ 6500 4200
 $Sheet
 S 7800 4000 850  400
@@
 Connection ~ 8800 4200
 $Comp
-L GND #PWR105
+L GND #PWR5
 U 1 1 53255562
 P 6300 4800
-F 0 "#PWR105" H 6300 4800 30  0001 C CNN
+F 0 "#PWR5" H 6300 4800 30  0001 C CNN
 F 1 "GND" H 6300 4730 30  0001 C CNN
 F 2 "" H 6300 4800 60  0000 C CNN
@@
 Connection ~ 8900 4200
 Wire Wire Line
-	6450 3500 7200 3500
-Wire Wire Line
-	8650 4200 9850 4200
-Wire Wire Line
-	10350 4200 11200 4200
+	6500 3500 7200 3500
+Wire Wire Line
+	8650 4200 9450 4200
 Wire Notes Line
 	6050 2800 9050 2800
@@
 	10650 3400 13150 3400
 Wire Notes Line
-	10650 5750 13150 5750
-Wire Notes Line
-	10650 5750 10650 3400
+	10650 5950 13150 5950
+Wire Notes Line
+	10650 5950 10650 3400
 Text Notes 10650 3375 0    60   ~ 0
 Voltage Limiting
@@
 Status LED
 Wire Notes Line
-	13150 5750 13150 3400
+	13150 5950 13150 3400
 Wire Wire Line
 	11800 4200 13600 4200
@@
 L R_0W25_1PCT R103
 U 1 1 5325DB3F
-P 12050 4550
-F 0 "R103" V 12130 4550 40  0000 C CNN
-F 1 "330" V 12057 4551 40  0000 C CNN
-F 2 "~" V 11980 4550 30  0000 C CNN
-F 3 "~" H 12050 4550 30  0000 C CNN
-	1    12050 4550
+P 12200 4550
+F 0 "R103" V 12280 4550 40  0000 C CNN
+F 1 "330" V 12207 4551 40  0000 C CNN
+F 2 "~" V 12130 4550 30  0000 C CNN
+F 3 "~" H 12200 4550 30  0000 C CNN
+	1    12200 4550
 	1    0    0    -1
 $EndComp
@@
 Connection ~ 13450 4200
 Wire Wire Line
-	6450 3500 6450 4200
-Text Notes 12300 5200 0    40   ~ 0
-330 & 5k = 20.2V max\n330 = 3.8mA error
-$Comp
-L GND #PWR106
+	6500 3500 6500 4200
+Text Notes 12150 4000 0    40   ~ 0
+330 & 5k = 20.2V max\n330 = 3.8mA ammeter error
+$Comp
+L GND #PWR6
 U 1 1 53264209
 P 6750 6700
-F 0 "#PWR106" H 6750 6700 30  0001 C CNN
+F 0 "#PWR6" H 6750 6700 30  0001 C CNN
 F 1 "GND" H 6750 6630 30  0001 C CNN
 F 2 "" H 6750 6700 60  0000 C CNN
@@
 $EndComp
 $Comp
-L GND #PWR107
+L GND #PWR7
 U 1 1 532642AB
 P 7250 6900
-F 0 "#PWR107" H 7250 6900 30  0001 C CNN
+F 0 "#PWR7" H 7250 6900 30  0001 C CNN
 F 1 "GND" H 7250 6830 30  0001 C CNN
 F 2 "" H 7250 6900 60  0000 C CNN
@@
 	5800 6300 6450 6300
 $Comp
-L GND #PWR104
+L GND #PWR4
 U 1 1 5326496C
 P 6250 6900
-F 0 "#PWR104" H 6250 6900 30  0001 C CNN
+F 0 "#PWR4" H 6250 6900 30  0001 C CNN
 F 1 "GND" H 6250 6830 30  0001 C CNN
 F 2 "" H 6250 6900 60  0000 C CNN
@@
 $EndComp
 $Comp
-L GND #PWR113
+L GND #PWR13
 U 1 1 5326745C
 P 13500 3200
-F 0 "#PWR113" H 13500 3200 30  0001 C CNN
+F 0 "#PWR13" H 13500 3200 30  0001 C CNN
 F 1 "GND" H 13500 3130 30  0001 C CNN
 F 2 "" H 13500 3200 60  0000 C CNN
@@
 5V
 $Comp
-L GND #PWR108
+L GND #PWR8
 U 1 1 53267BC5
 P 9350 4100
-F 0 "#PWR108" H 9350 4100 30  0001 C CNN
+F 0 "#PWR8" H 9350 4100 30  0001 C CNN
 F 1 "GND" H 9350 4030 30  0001 C CNN
 F 2 "" H 9350 4100 60  0000 C CNN
@@
 Connection ~ 4700 4200
 Wire Wire Line
-	12000 4200 12000 3750
-Wire Wire Line
-	12000 3750 11700 3750
-Wire Wire Line
-	11300 3750 11000 3750
-Wire Wire Line
-	11000 3750 11000 4200
-Connection ~ 11000 4200
+	12050 4200 12050 3850
+Wire Wire Line
+	12050 3850 11700 3850
+Wire Wire Line
+	11300 3850 11050 3850
+Wire Wire Line
+	11050 3850 11050 4200
+Connection ~ 11050 4200
 Wire Wire Line
 	4300 4300 4300 4200
@@
 	7650 3800 7650 4200
 Wire Wire Line
-	6950 3800 6650 3800
-Wire Wire Line
-	6650 3800 6650 4200
-Connection ~ 6650 4200
+	6950 3800 6700 3800
+Wire Wire Line
+	6700 3800 6700 4200
+Connection ~ 6700 4200
 Wire Wire Line
 	6300 4300 6300 4200
@@
 P 4300 4500
 F 0 "C102" H 4320 4560 30  0000 L BNN
-F 1 "1000uF" H 4320 4410 30  0000 L TNN
+F 1 "100uF" H 4320 4410 30  0000 L TNN
 F 2 "~" H 4338 4350 30  0000 C CNN
 F 3 "~" H 4300 4500 60  0000 C CNN
@@
 L C_EL C104
 U 1 1 53268E70
-P 11500 5200
-F 0 "C104" H 11520 5260 30  0000 L BNN
-F 1 "10uF" H 11520 5110 30  0000 L TNN
-F 2 "~" H 11538 5050 30  0000 C CNN
-F 3 "~" H 11500 5200 60  0000 C CNN
-	1    11500 5200
+P 12500 5450
+F 0 "C104" H 12520 5510 30  0000 L BNN
+F 1 "10uF" H 12520 5360 30  0000 L TNN
+F 2 "~" H 12538 5300 30  0000 C CNN
+F 3 "~" H 12500 5450 60  0000 C CNN
+	1    12500 5450
 	1    0    0    -1
 $EndComp
@@
 	0    1    1    0
 $EndComp
+$Comp
+L DIODE D1
+U 1 1 5327B26B
+P 7550 4550
+F 0 "D1" H 7550 4650 40  0000 C CNN
+F 1 "1N4148" H 7550 4450 40  0000 C CNN
+F 2 "~" H 7550 4550 60  0000 C CNN
+F 3 "~" H 7550 4550 60  0000 C CNN
+	1    7550 4550
+	0    -1   -1   0
+$EndComp
+Wire Wire Line
+	7550 4350 7550 4200
+Connection ~ 7550 4200
+Wire Wire Line
+	7550 4750 7550 4850
+Wire Wire Line
+	7550 4850 7150 4850
+Connection ~ 7150 4850
+Wire Wire Line
+	12200 4300 12200 4200
+Wire Wire Line
+	11900 4300 11900 4200
+Wire Wire Line
+	11900 4700 11900 4750
+Wire Wire Line
+	11900 4750 11500 4750
+Connection ~ 11500 4750
+Wire Wire Line
+	12200 4800 12200 5150
+Wire Wire Line
+	12200 5750 12200 5650
+Connection ~ 12200 4900
+Wire Wire Line
+	12500 5650 12500 5750
+Wire Wire Line
+	11500 4500 11500 4900
+Wire Wire Line
+	12200 5100 12000 5100
+Wire Wire Line
+	12000 5100 12000 5400
+Wire Wire Line
+	12000 5400 12050 5400
+Connection ~ 12200 5100
+Wire Wire Line
+	12500 5250 12500 5000
+Wire Wire Line
+	12500 5000 12200 5000
+Connection ~ 12200 5000
+Wire Wire Line
+	10350 4200 11200 4200
 $EndSCHEMATC

Commit message: moving status LED to 5V rail.  starting initial layout.
Parts:
- R101: value 1k -> 150
Connections:
- wire segments 80 -> 102
Other:
- moved on the sheet: C101, C102, C103, C104, C105, C106, C107, CON101, D1, D101, D102, D103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

Commit message: updating schematic
Connections:
- wire segments 102 -> 78
Changed lines of the file:
@@
 	6100 5150 7750 5150
 Wire Wire Line
-	6100 4650 6100 5000
-Wire Wire Line
-	6100 5000 6100 5150
+	6100 4650 6100 5150
 Wire Wire Line
 	7550 7500 7550 7600
@@
 $EndSheet
 Wire Wire Line
-	6400 4350 6500 4350
-Wire Wire Line
-	6500 4350 6600 4350
-Wire Wire Line
-	6600 4350 6750 4350
+	6400 4350 6750 4350
 Connection ~ 6600 4350
 Wire Wire Line
@@
 	6800 3550 7850 3550
 Wire Wire Line
-	7850 3550 7850 4350
+	7850 4350 7850 3550
 Connection ~ 7850 4350
 Wire Wire Line
 	5450 3650 6150 3650
 Wire Wire Line
-	7600 4350 7750 4350
-Wire Wire Line
-	7750 4350 7850 4350
-Wire Wire Line
-	7850 4350 8400 4350
+	7600 4350 8400 4350
 Wire Notes Line
 	5000 2950 8000 2950
@@
 	12100 6100 12100 3550
 Wire Wire Line
-	10750 4350 10850 4350
-Wire Wire Line
-	10850 4350 11000 4350
-Wire Wire Line
-	11000 4350 11150 4350
-Wire Wire Line
-	11150 4350 11750 4350
-Wire Wire Line
-	11750 4350 12400 4350
-Wire Wire Line
-	12400 4350 12550 4350
+	10750 4350 12550 4350
 $Comp
 L R_0W25_1PCT R103
@@
 	4100 4250 4100 4350
 Wire Wire Line
-	4100 4350 4450 4350
-Wire Wire Line
-	4450 4350 4750 4350
-Wire Wire Line
-	4750 4350 5250 4350
-Wire Wire Line
-	5250 4350 5450 4350
-Wire Wire Line
-	5450 4350 5650 4350
-Wire Wire Line
-	5650 4350 5800 4350
+	4100 4350 5800 4350
 Text Notes 3450 4150 0    40   ~ 0
 Power On / Off
@@
 	6200 6550 6200 6450
 Wire Wire Line
-	6000 6450 6200 6450
-Wire Wire Line
-	6200 6450 6300 6450
+	6000 6450 6300 6450
 Wire Wire Line
 	6300 6450 6300 6350
@@
 5V
 Wire Wire Line
-	4750 6450 5200 6450
-Wire Wire Line
-	5200 6450 5400 6450
+	4750 6450 5400 6450
 $Comp
 L GND #PWR012
@@
 	10250 4000 10000 4000
 Wire Wire Line
-	10000 4000 10000 4350
+	10000 4350 10000 4000
 Connection ~ 10000 4350
 Wire Wire Line
@@
 	2650 4450 2750 4450
 Wire Wire Line
-	2750 4450 2750 4550
-Wire Wire Line
-	2750 4550 2750 4650
+	2750 4450 2750 4650
 Wire Wire Line
 	2650 4550 2750 4550
@@
 Connection ~ 10450 4900
 Wire Wire Line
-	11150 4950 11150 5050
-Wire Wire Line
-	11150 5050 11150 5150
-Wire Wire Line
-	11150 5150 11150 5250
-Wire Wire Line
-	11150 5250 11150 5300
+	11150 4950 11150 5300
 Wire Wire Line
 	11150 5900 11150 5800
@@
 	11450 5800 11450 5900
 Wire Wire Line
-	10450 4650 10450 4900
-Wire Wire Line
-	10450 4900 10450 5050
+	10450 4650 10450 5050
 Wire Wire Line
 	11150 5250 10950 5250
@@
 Connection ~ 11150 5150
 Wire Wire Line
-	9300 4350 9800 4350
-Wire Wire Line
-	9800 4350 10000 4350
-Wire Wire Line
-	10000 4350 10150 4350
+	9300 4350 10150 4350
 Text GLabel 7550 6400 1    40   Input ~ 0
 5V

Commit message: reconfiguring ammeter to be low-side, not high-side.
Parts:
- removed DS101: AMMETER, ~, symbol AMMETER
- removed U101: 7805, ~, symbol 7805
- added C?: 0.1uF, ~, symbol C_CER
- added C?: 10uF, ~, symbol C_EL
- added DS?: AMMETER_V, ~, symbol AMMETER_V
- added U? (x2): 78L05, ~, symbol 78L05
Connections:
- net labels added: 5VF, Vout-
- wire segments 78 -> 92
Other:
- note added: "5VF Supply"
- moved on the sheet: C101, C102, C103, C104, C105, C106, C107, CON101, D1, D101, D102, D103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

Commit message: switching to voltmeter based on real ground, not Vout- (introduced too much error into the ammeter)
Parts:
- removed C?: 0.1uF, ~, symbol C_CER
- removed C?: 10uF, ~, symbol C_EL
- removed U?: 78L05, ~, symbol 78L05
- RV101: value 5k -> 4k7
Connections:
- net labels removed: 5VF, Vout-
- wire segments 92 -> 80
Other:
- note added: "330 & 4.7k = 19V max"
- note removed: "330 & 5k = 20.2V max\n330 = 3.8mA ammeter error"
- note removed: "5VF Supply"
Changed lines of the file:
@@
 Sheet 1 2
 Title ""
-Date "20 mar 2014"
+Date "21 mar 2014"
 Rev ""
 Comp ""
@@
 P 10650 5400
 F 0 "RV101" H 10650 5300 50  0000 C CNN
-F 1 "5k" H 10650 5400 50  0000 C CNN
+F 1 "4k7" H 10650 5400 50  0000 C CNN
 F 2 "~" H 10650 5400 60  0000 C CNN
 F 3 "~" H 10650 5400 60  0000 C CNN
@@
 Wire Wire Line
 	6050 3500 6050 4200
-Text Notes 10600 4000 0    40   ~ 0
-330 & 5k = 20.2V max\n330 = 3.8mA ammeter error
+Text Notes 9850 5050 0    40   ~ 0
+330 & 4.7k = 19V max
 $Comp
 L GND #PWR010
@@
 	1    0    0    -1
 $EndComp
-Wire Wire Line
-	11850 3100 12050 3100
-Wire Wire Line
-	12050 3000 11950 3000
-Wire Wire Line
-	11950 3000 11950 2900
-Text GLabel 11950 2900 1    40   Input ~ 0
-5VF
+Text GLabel 11850 2900 1    40   Input ~ 0
+5V
 $Comp
 L GND #PWR014
@@
 Wire Wire Line
 	11950 3300 11950 4200
-Wire Wire Line
-	5350 4200 5350 7850
 Connection ~ 5350 4200
 Wire Wire Line
@@
 Wire Wire Line
 	13050 5650 13050 5950
-Text GLabel 12950 4800 3    40   Input ~ 0
-Vout-
-Text GLabel 11850 3200 3    40   Input ~ 0
-Vout-
-Wire Wire Line
-	6800 7950 6800 7850
-Wire Wire Line
-	6600 7850 6900 7850
-Wire Wire Line
-	6900 7850 6900 7750
-Connection ~ 6800 7850
-Text GLabel 6900 7750 1    40   Input ~ 0
-5VF
-Wire Wire Line
-	5350 7850 6000 7850
-Wire Wire Line
-	5800 7950 5800 7850
-Connection ~ 5800 7850
-Wire Notes Line
-	5600 7500 7150 7500
-Wire Notes Line
-	7150 7500 7150 8900
-Wire Notes Line
-	7150 8900 5600 8900
-Wire Notes Line
-	5600 8900 5600 7500
-Text Notes 5600 7475 0    60   ~ 0
-5VF Supply
-$Comp
-L C_CER C?
-U 1 1 532A79E0
-P 5800 8150
-F 0 "C?" H 5820 8210 30  0000 L BNN
-F 1 "0.1uF" H 5820 8090 30  0000 L TNN
-F 2 "~" H 5838 8000 30  0000 C CNN
-F 3 "~" H 5800 8150 60  0000 C CNN
-	1    5800 8150
-	1    0    0    -1
-$EndComp
-$Comp
-L C_EL C?
-U 1 1 532A79E6
-P 6800 8150
-F 0 "C?" H 6820 8210 30  0000 L BNN
-F 1 "10uF" H 6820 8060 30  0000 L TNN
-F 2 "~" H 6838 8000 30  0000 C CNN
-F 3 "~" H 6800 8150 60  0000 C CNN
-	1    6800 8150
-	1    0    0    -1
-$EndComp
-$Comp
-L 78L05 U?
-U 1 1 532A7B70
-P 6300 7900
-F 0 "U?" H 6100 8060 40  0000 L BNN
-F 1 "78L05" H 6500 7730 40  0000 R TNN
-F 2 "~" H 6300 7900 60  0000 C CNN
-F 3 "~" H 6300 7900 60  0000 C CNN
-	1    6300 7900
-	1    0    0    -1
-$EndComp
 $Comp
 L 78L05 U?
@@
 	1    0    0    -1
 $EndComp
-Text GLabel 6400 8550 3    40   Input ~ 0
-Vout-
-Wire Wire Line
-	5800 8350 5800 8450
-Wire Wire Line
-	5800 8450 6800 8450
-Wire Wire Line
-	6800 8450 6800 8350
-Wire Wire Line
-	6300 8150 6300 8450
-Connection ~ 6300 8450
-Wire Wire Line
-	6400 8450 6400 8550
-Connection ~ 6400 8450
-Connection ~ 5350 6300
-Wire Wire Line
-	13050 4700 12950 4700
-Wire Wire Line
-	12950 4700 12950 4800
-Connection ~ 13050 4700
+$Comp
+L GND #PWR?
+U 1 1 532B868B
+P 11850 3200
+F 0 "#PWR?" H 11850 3200 30  0001 C CNN
+F 1 "GND" H 11850 3130 30  0001 C CNN
+F 2 "" H 11850 3200 60  0000 C CNN
+F 3 "" H 11850 3200 60  0000 C CNN
+	1    11850 3200
+	1    0    0    -1
+$EndComp
+Wire Wire Line
+	12050 3100 11850 3100
 Wire Wire Line
 	11850 3100 11850 3200
+Wire Wire Line
+	12050 3000 11850 3000
+Wire Wire Line
+	11850 3000 11850 2900
+Wire Wire Line
+	5350 6300 5350 4200
 $EndSCHEMATC
