File: DualLM317BenchSupply/DualLM317BenchSupply.sch (KiCad schematic (older format))
At the start: 26 parts, among them CON101 BARREL_JACK, P103 CONN_1, P104 CONN_1, SW101 SPDT, SW102 SPDT, SW103 SPDT, U102 LM317, U103 LM317

Commit message: specifying 1% for current limiting resistors (lower temp co).  also, moving 10R resistors to 1/2 watt.
Parts:
- gave numbers to parts that had none: 2
- renumbered C102 to C101, C106 to C102, C101 to C103, C107 to C104, C103 to C105, C104 to C106, C105 to C107, D104 to D101, D1 to D102, D101 to D103, D102 to D104, D103 to D105, DS102 to DS101, P103 to P101, P104 to P102, R103 to R102
Changed lines of the file:
@@
 Sheet 1 2
 Title ""
-Date "21 mar 2014"
+Date "22 mar 2014"
 Rev ""
 Comp ""
@@
 $EndDescr
 $Comp
-L GND #PWR01
+L GND #PWR107
 U 1 1 5311570D
 P 8150 7450
-F 0 "#PWR01" H 8150 7450 30  0001 C CNN
+F 0 "#PWR107" H 8150 7450 30  0001 C CNN
 F 1 "GND" H 8150 7380 30  0001 C CNN
 F 2 "" H 8150 7450 60  0000 C CNN
@@
 $EndComp
 $Comp
-L GND #PWR02
+L GND #PWR108
 U 1 1 5311577C
 P 9300 4800
-F 0 "#PWR02" H 9300 4800 30  0001 C CNN
+F 0 "#PWR108" H 9300 4800 30  0001 C CNN
 F 1 "GND" H 9300 4730 30  0001 C CNN
 F 2 "" H 9300 4800 60  0000 C CNN
@@
 $EndComp
 $Comp
-L GND #PWR03
+L GND #PWR102
 U 1 1 531157E6
 P 5050 4800
-F 0 "#PWR03" H 5050 4800 30  0001 C CNN
+F 0 "#PWR102" H 5050 4800 30  0001 C CNN
 F 1 "GND" H 5050 4730 30  0001 C CNN
 F 2 "" H 5050 4800 60  0000 C CNN
@@
 $EndComp
 $Comp
-L GND #PWR04
+L GND #PWR109
 U 1 1 53116107
 P 10650 5750
-F 0 "#PWR04" H 10650 5750 30  0001 C CNN
+F 0 "#PWR109" H 10650 5750 30  0001 C CNN
 F 1 "GND" H 10650 5680 30  0001 C CNN
 F 2 "" H 10650 5750 60  0000 C CNN
@@
 $EndComp
 $Comp
-L GND #PWR05
+L GND #PWR110
 U 1 1 53116125
 P 10950 5750
-F 0 "#PWR05" H 10950 5750 30  0001 C CNN
+F 0 "#PWR110" H 10950 5750 30  0001 C CNN
 F 1 "GND" H 10950 5680 30  0001 C CNN
 F 2 "" H 10950 5750 60  0000 C CNN
@@
 $EndComp
 $Comp
-L DIODE D103
+L DIODE D105
 U 1 1 53116214
 P 10350 4500
-F 0 "D103" H 10350 4600 40  0000 C CNN
+F 0 "D105" H 10350 4600 40  0000 C CNN
 F 1 "1N4148" H 10350 4400 40  0000 C CNN
 F 2 "~" H 10350 4500 60  0000 C CNN
@@
 $EndComp
 $Comp
-L DIODE D102
+L DIODE D104
 U 1 1 53116272
 P 9950 3850
-F 0 "D102" H 9950 3950 40  0000 C CNN
+F 0 "D104" H 9950 3950 40  0000 C CNN
 F 1 "1N4148" H 9950 3750 40  0000 C CNN
 F 2 "~" H 9950 3850 60  0000 C CNN
@@
 Connection ~ 11250 4200
 $Comp
-L GND #PWR06
+L GND #PWR111
 U 1 1 531163B7
 P 11250 4800
-F 0 "#PWR06" H 11250 4800 30  0001 C CNN
+F 0 "#PWR111" H 11250 4800 30  0001 C CNN
 F 1 "GND" H 11250 4730 30  0001 C CNN
 F 2 "" H 11250 4800 60  0000 C CNN
@@
 Current Limit Bypass
 $Comp
-L CONN_1 P103
+L CONN_1 P101
 U 1 1 5311679A
 P 13300 4200
-F 0 "P103" H 13380 4200 40  0000 L CNN
+F 0 "P101" H 13380 4200 40  0000 L CNN
 F 1 "CONN_1" H 13300 4255 30  0001 C CNN
 F 2 "" H 13300 4200 60  0000 C CNN
@@
 $EndComp
 $Comp
-L CONN_1 P104
+L CONN_1 P102
 U 1 1 531167A9
 P 13300 4600
-F 0 "P104" H 13380 4600 40  0000 L CNN
+F 0 "P102" H 13380 4600 40  0000 L CNN
 F 1 "CONN_1" H 13300 4655 30  0001 C CNN
 F 2 "" H 13300 4600 60  0000 C CNN
@@
 $EndComp
 $Comp
-L GND #PWR07
+L GND #PWR114
 U 1 1 53116825
 P 13050 5950
-F 0 "#PWR07" H 13050 5950 30  0001 C CNN
+F 0 "#PWR114" H 13050 5950 30  0001 C CNN
 F 1 "GND" H 13050 5880 30  0001 C CNN
 F 2 "" H 13050 5950 60  0000 C CNN
@@
 Vout\n(1.25V - 20.2V DC)
 $Comp
-L GND #PWR08
+L GND #PWR101
 U 1 1 53116888
 P 3350 4500
-F 0 "#PWR08" H 3350 4500 30  0001 C CNN
+F 0 "#PWR101" H 3350 4500 30  0001 C CNN
 F 1 "GND" H 3350 4430 30  0001 C CNN
 F 2 "" H 3350 4500 60  0000 C CNN
@@
 Connection ~ 8350 4200
 $Comp
-L GND #PWR09
+L GND #PWR104
 U 1 1 53255562
 P 5850 4800
-F 0 "#PWR09" H 5850 4800 30  0001 C CNN
+F 0 "#PWR104" H 5850 4800 30  0001 C CNN
 F 1 "GND" H 5850 4730 30  0001 C CNN
 F 2 "" H 5850 4800 60  0000 C CNN
@@
 	10250 4200 12050 4200
 $Comp
-L R_0W25_1PCT R103
+L R_0W25_1PCT R102
 U 1 1 5325DB3F
 P 10650 4550
-F 0 "R103" V 10730 4550 40  0000 C CNN
+F 0 "R102" V 10730 4550 40  0000 C CNN
 F 1 "330" V 10657 4551 40  0000 C CNN
 F 2 "~" V 10580 4550 30  0000 C CNN
@@
 330 & 4.7k = 19V max
 $Comp
-L GND #PWR010
+L GND #PWR105
 U 1 1 53264209
 P 6300 6700
-F 0 "#PWR010" H 6300 6700 30  0001 C CNN
+F 0 "#PWR105" H 6300 6700 30  0001 C CNN
 F 1 "GND" H 6300 6630 30  0001 C CNN
 F 2 "" H 6300 6700 60  0000 C CNN
@@
 $EndComp
 $Comp
-L GND #PWR011
+L GND #PWR106
 U 1 1 532642AB
 P 6800 6900
-F 0 "#PWR011" H 6800 6900 30  0001 C CNN
+F 0 "#PWR106" H 6800 6900 30  0001 C CNN
 F 1 "GND" H 6800 6830 30  0001 C CNN
 F 2 "" H 6800 6900 60  0000 C CNN
@@
 	5350 6300 6000 6300
 $Comp
-L GND #PWR012
+L GND #PWR103
 U 1 1 5326496C
 P 5800 6900
-F 0 "#PWR012" H 5800 6900 30  0001 C CNN
+F 0 "#PWR103" H 5800 6900 30  0001 C CNN
 F 1 "GND" H 5800 6830 30  0001 C CNN
 F 2 "" H 5800 6900 60  0000 C CNN
@@
 5V Supply
 $Comp
-L VOLTMETER DS102
+L VOLTMETER DS101
 U 1 1 53267314
 P 12050 3000
-F 0 "DS102" H 12100 3150 40  0000 L CNN
+F 0 "DS101" H 12100 3150 40  0000 L CNN
 F 1 "VOLTMETER" H 12900 2600 40  0000 R CNN
 F 2 "~" H 12880 3400 60  0000 C CNN
@@
 5V
 $Comp
-L GND #PWR014
+L GND #PWR113
 U 1 1 53267BC5
 P 11950 5550
-F 0 "#PWR014" H 11950 5550 30  0001 C CNN
+F 0 "#PWR113" H 11950 5550 30  0001 C CNN
 F 1 "GND" H 11950 5480 30  0001 C CNN
 F 2 "" H 11950 5550 60  0000 C CNN
@@
 Connection ~ 5050 4200
 $Comp
-L DIODE D104
+L DIODE D101
 U 1 1 53265FE1
 P 6700 3800
-F 0 "D104" H 6700 3900 40  0000 C CNN
+F 0 "D101" H 6700 3900 40  0000 C CNN
 F 1 "1N4148" H 6700 3700 40  0000 C CNN
 F 2 "~" H 6700 3800 60  0000 C CNN
@@
 $EndComp
 $Comp
-L C_CER C106
+L C_CER C102
 U 1 1 53268218
 P 5800 6600
-F 0 "C106" H 5820 6660 30  0000 L BNN
+F 0 "C102" H 5820 6660 30  0000 L BNN
 F 1 "0.1uF" H 5820 6540 30  0000 L TNN
 F 2 "~" H 5838 6450 30  0000 C CNN
@@
 $EndComp
 $Comp
-L C_EL C107
+L C_EL C104
 U 1 1 53268227
 P 6800 6600
-F 0 "C107" H 6820 6660 30  0000 L BNN
+F 0 "C104" H 6820 6660 30  0000 L BNN
 F 1 "10uF" H 6820 6510 30  0000 L TNN
 F 2 "~" H 6838 6450 30  0000 C CNN
@@
 $EndComp
 $Comp
-L C_EL C102
+L C_EL C101
 U 1 1 53268786
 P 5050 4500
-F 0 "C102" H 5070 4560 30  0000 L BNN
+F 0 "C101" H 5070 4560 30  0000 L BNN
 F 1 "100uF" H 5070 4410 30  0000 L TNN
 F 2 "~" H 5088 4350 30  0000 C CNN
@@
 $EndComp
 $Comp
-L C_CER C101
+L C_CER C103
 U 1 1 53268930
 P 5850 4500
-F 0 "C101" H 5870 4560 30  0000 L BNN
+F 0 "C103" H 5870 4560 30  0000 L BNN
 F 1 "0.1uF" H 5870 4440 30  0000 L TNN
 F 2 "~" H 5888 4350 30  0000 C CNN
@@
 $EndComp
 $Comp
-L C_EL C103
+L C_EL C105
 U 1 1 53268CD2
 P 9300 4500
-F 0 "C103" H 9320 4560 30  0000 L BNN
+F 0 "C105" H 9320 4560 30  0000 L BNN
 F 1 "1uF" H 9320 4410 30  0000 L TNN
 F 2 "~" H 9338 4350 30  0000 C CNN
@@
 $EndComp
 $Comp
-L C_EL C104
+L C_EL C106
 U 1 1 53268E70
 P 10950 5450
-F 0 "C104" H 10970 5510 30  0000 L BNN
+F 0 "C106" H 10970 5510 30  0000 L BNN
 F 1 "10uF" H 10970 5360 30  0000 L TNN
 F 2 "~" H 10988 5300 30  0000 C CNN
@@
 $EndComp
 $Comp
-L C_EL C105
+L C_EL C107
 U 1 1 53269020
 P 11250 4500
-F 0 "C105" H 11270 4560 30  0000 L BNN
+F 0 "C107" H 11270 4560 30  0000 L BNN
 F 1 "1uF" H 11270 4410 30  0000 L TNN
 F 2 "~" H 11288 4350 30  0000 C CNN
@@
 $EndComp
 $Comp
-L LED D101
+L LED D103
 U 1 1 5326B9A5
 P 8150 6550
-F 0 "D101" H 8025 6650 40  0000 C CNN
+F 0 "D103" H 8025 6650 40  0000 C CNN
 F 1 "LED" H 8275 6650 30  0000 C CNN
 F 2 "~" H 8150 6550 60  0000 C CNN
@@
 $EndComp
 $Comp
-L DIODE D1
+L DIODE D102
 U 1 1 5327B26B
 P 7100 4550
-F 0 "D1" H 7100 4650 40  0000 C CNN
+F 0 "D102" H 7100 4650 40  0000 C CNN
 F 1 "1N4148" H 7100 4450 40  0000 C CNN
 F 2 "~" H 7100 4550 60  0000 C CNN
@@
 5V
 $Comp
-L AMMETER_V DS?
+L AMMETER_V DS102
 U 1 1 532A6A61
 P 12050 5350
-F 0 "DS?" H 12100 5500 40  0000 L CNN
+F 0 "DS102" H 12100 5500 40  0000 L CNN
 F 1 "AMMETER_V" H 12900 4950 40  0000 R CNN
 F 2 "~" H 12880 5750 60  0000 C CNN
@@
 	13050 5650 13050 5950
 $Comp
-L 78L05 U?
+L 78L05 U101
 U 1 1 532A7BBB
 P 6300 6350
-F 0 "U?" H 6100 6510 40  0000 L BNN
+F 0 "U101" H 6100 6510 40  0000 L BNN
 F 1 "78L05" H 6500 6180 40  0000 R TNN
 F 2 "~" H 6300 6350 60  0000 C CNN
@@
 $EndComp
 $Comp
-L GND #PWR?
+L GND #PWR112
 U 1 1 532B868B
 P 11850 3200
-F 0 "#PWR?" H 11850 3200 30  0001 C CNN
+F 0 "#PWR112" H 11850 3200 30  0001 C CNN
 F 1 "GND" H 11850 3130 30  0001 C CNN
 F 2 "" H 11850 3200 60  0000 C CNN
