File: DualLM317BenchSupply/DualLM317BenchSupply.sch (KiCad schematic (older format))
At the start: 26 parts, among them CON101 BARREL_JACK, P101 CONN_1, P102 CONN_1, SW101 SPDT, SW102 SPDT, SW103 SPDT, U101 78L05, U102 LM317, U103 LM317

Commit message: adding second dc jack
Parts:
- added CON102: BARREL_JACK, ~, symbol BARREL_JACK
Connections:
- wire segments 80 -> 85
Other:
- note added: "2.1 x 5.5mm"
- note added: "2.5 x 5.5mm"
Changed lines of the file:
@@
 Sheet 1 2
 Title ""
-Date "22 mar 2014"
+Date "23 mar 2014"
 Rev ""
 Comp ""
@@
 $EndDescr
 $Comp
-L GND #PWR01
+L GND #PWR108
 U 1 1 5311570D
 P 8150 7450
-F 0 "#PWR01" H 8150 7450 30  0001 C CNN
+F 0 "#PWR108" H 8150 7450 30  0001 C CNN
 F 1 "GND" H 8150 7380 30  0001 C CNN
 F 2 "" H 8150 7450 60  0000 C CNN
@@
 $EndComp
 $Comp
-L GND #PWR02
+L GND #PWR109
 U 1 1 5311577C
 P 9300 4800
-F 0 "#PWR02" H 9300 4800 30  0001 C CNN
+F 0 "#PWR109" H 9300 4800 30  0001 C CNN
 F 1 "GND" H 9300 4730 30  0001 C CNN
 F 2 "" H 9300 4800 60  0000 C CNN
@@
 $EndComp
 $Comp
-L GND #PWR03
+L GND #PWR103
 U 1 1 531157E6
 P 5050 4800
-F 0 "#PWR03" H 5050 4800 30  0001 C CNN
+F 0 "#PWR103" H 5050 4800 30  0001 C CNN
 F 1 "GND" H 5050 4730 30  0001 C CNN
 F 2 "" H 5050 4800 60  0000 C CNN
@@
 $EndComp
 $Comp
-L GND #PWR04
+L GND #PWR110
 U 1 1 53116107
 P 10650 5750
-F 0 "#PWR04" H 10650 5750 30  0001 C CNN
+F 0 "#PWR110" H 10650 5750 30  0001 C CNN
 F 1 "GND" H 10650 5680 30  0001 C CNN
 F 2 "" H 10650 5750 60  0000 C CNN
@@
 $EndComp
 $Comp
-L GND #PWR05
+L GND #PWR111
 U 1 1 53116125
 P 10950 5750
-F 0 "#PWR05" H 10950 5750 30  0001 C CNN
+F 0 "#PWR111" H 10950 5750 30  0001 C CNN
 F 1 "GND" H 10950 5680 30  0001 C CNN
 F 2 "" H 10950 5750 60  0000 C CNN
@@
 Connection ~ 11250 4200
 $Comp
-L GND #PWR06
+L GND #PWR112
 U 1 1 531163B7
 P 11250 4800
-F 0 "#PWR06" H 11250 4800 30  0001 C CNN
+F 0 "#PWR112" H 11250 4800 30  0001 C CNN
 F 1 "GND" H 11250 4730 30  0001 C CNN
 F 2 "" H 11250 4800 60  0000 C CNN
@@
 $EndComp
 $Comp
-L GND #PWR07
+L GND #PWR115
 U 1 1 53116825
 P 13050 5950
-F 0 "#PWR07" H 13050 5950 30  0001 C CNN
+F 0 "#PWR115" H 13050 5950 30  0001 C CNN
 F 1 "GND" H 13050 5880 30  0001 C CNN
 F 2 "" H 13050 5950 60  0000 C CNN
@@
 Vout\n(1.25V - 20.2V DC)
 $Comp
-L GND #PWR08
+L GND #PWR101
 U 1 1 53116888
 P 3350 4500
-F 0 "#PWR08" H 3350 4500 30  0001 C CNN
+F 0 "#PWR101" H 3350 4500 30  0001 C CNN
 F 1 "GND" H 3350 4430 30  0001 C CNN
 F 2 "" H 3350 4500 60  0000 C CNN
@@
 Connection ~ 8350 4200
 $Comp
-L GND #PWR09
+L GND #PWR105
 U 1 1 53255562
 P 5850 4800
-F 0 "#PWR09" H 5850 4800 30  0001 C CNN
+F 0 "#PWR105" H 5850 4800 30  0001 C CNN
 F 1 "GND" H 5850 4730 30  0001 C CNN
 F 2 "" H 5850 4800 60  0000 C CNN
@@
 330 & 4.7k = 19V max
 $Comp
-L GND #PWR010
+L GND #PWR106
 U 1 1 53264209
 P 6300 6700
-F 0 "#PWR010" H 6300 6700 30  0001 C CNN
+F 0 "#PWR106" H 6300 6700 30  0001 C CNN
 F 1 "GND" H 6300 6630 30  0001 C CNN
 F 2 "" H 6300 6700 60  0000 C CNN
@@
 $EndComp
 $Comp
-L GND #PWR011
+L GND #PWR107
 U 1 1 532642AB
 P 6800 6900
-F 0 "#PWR011" H 6800 6900 30  0001 C CNN
+F 0 "#PWR107" H 6800 6900 30  0001 C CNN
 F 1 "GND" H 6800 6830 30  0001 C CNN
 F 2 "" H 6800 6900 60  0000 C CNN
@@
 	5350 6300 6000 6300
 $Comp
-L GND #PWR012
+L GND #PWR104
 U 1 1 5326496C
 P 5800 6900
-F 0 "#PWR012" H 5800 6900 30  0001 C CNN
+F 0 "#PWR104" H 5800 6900 30  0001 C CNN
 F 1 "GND" H 5800 6830 30  0001 C CNN
 F 2 "" H 5800 6900 60  0000 C CNN
@@
 5V
 $Comp
-L GND #PWR013
+L GND #PWR114
 U 1 1 53267BC5
 P 11950 5550
-F 0 "#PWR013" H 11950 5550 30  0001 C CNN
+F 0 "#PWR114" H 11950 5550 30  0001 C CNN
 F 1 "GND" H 11950 5480 30  0001 C CNN
 F 2 "" H 11950 5550 60  0000 C CNN
@@
 $EndComp
 $Comp
-L GND #PWR014
+L GND #PWR113
 U 1 1 532B868B
 P 11850 3200
-F 0 "#PWR014" H 11850 3200 30  0001 C CNN
+F 0 "#PWR113" H 11850 3200 30  0001 C CNN
 F 1 "GND" H 11850 3130 30  0001 C CNN
 F 2 "" H 11850 3200 60  0000 C CNN
@@
 Wire Wire Line
 	5350 6300 5350 4200
+$Comp
+L BARREL_JACK CON102
+U 1 1 532F003E
+P 2950 4900
+F 0 "CON102" H 2950 5100 40  0000 C CNN
+F 1 "BARREL_JACK" H 2950 4750 40  0000 C CNN
+F 2 "~" H 2950 4900 60  0000 C CNN
+F 3 "~" H 2950 4900 60  0000 C CNN
+	1    2950 4900
+	1    0    0    -1
+$EndComp
+$Comp
+L GND #PWR102
+U 1 1 532F0044
+P 3350 5100
+F 0 "#PWR102" H 3350 5100 30  0001 C CNN
+F 1 "GND" H 3350 5030 30  0001 C CNN
+F 2 "" H 3350 5100 60  0000 C CNN
+F 3 "" H 3350 5100 60  0000 C CNN
+	1    3350 5100
+	1    0    0    -1
+$EndComp
+Wire Wire Line
+	3250 4900 3350 4900
+Wire Wire Line
+	3350 4900 3350 5100
+Wire Wire Line
+	3250 5000 3350 5000
+Connection ~ 3350 5000
+Wire Wire Line
+	3250 4800 3450 4800
+Wire Wire Line
+	3450 4800 3450 4200
+Connection ~ 3450 4200
+Text Notes 2150 4250 0    40   ~ 0
+2.1 x 5.5mm
+Text Notes 2150 4850 0    40   ~ 0
+2.5 x 5.5mm
 $EndSCHEMATC

Commit message: adding mounting holes to schematic
Parts:
- added H101, H102, H103, H104: HOLE, ~, symbol HOLE
Changed lines of the file:
@@
 EESchema Schematic File Version 2
+LIBS:mounting_holes_PL
 LIBS:LEDs_PL
 LIBS:regulators_PL
@@
 Text Notes 2150 4850 0    40   ~ 0
 2.5 x 5.5mm
+$Comp
+L HOLE H101
+U 1 1 532F0654
+P 650 10350
+F 0 "H101" H 650 10405 30  0000 C CNN
+F 1 "HOLE" H 650 10290 30  0000 C CNN
+F 2 "~" H 650 10350 60  0000 C CNN
+F 3 "~" H 650 10350 60  0000 C CNN
+	1    650  10350
+	1    0    0    -1
+$EndComp
+$Comp
+L HOLE H102
+U 1 1 532F0663
+P 850 10350
+F 0 "H102" H 850 10405 30  0000 C CNN
+F 1 "HOLE" H 850 10290 30  0000 C CNN
+F 2 "~" H 850 10350 60  0000 C CNN
+F 3 "~" H 850 10350 60  0000 C CNN
+	1    850  10350
+	1    0    0    -1
+$EndComp
+$Comp
+L HOLE H103
+U 1 1 532F0672
+P 1050 10350
+F 0 "H103" H 1050 10405 30  0000 C CNN
+F 1 "HOLE" H 1050 10290 30  0000 C CNN
+F 2 "~" H 1050 10350 60  0000 C CNN
+F 3 "~" H 1050 10350 60  0000 C CNN
+	1    1050 10350
+	1    0    0    -1
+$EndComp
+$Comp
+L HOLE H104
+U 1 1 532F0681
+P 1250 10350
+F 0 "H104" H 1250 10405 30  0000 C CNN
+F 1 "HOLE" H 1250 10290 30  0000 C CNN
+F 2 "~" H 1250 10350 60  0000 C CNN
+F 3 "~" H 1250 10350 60  0000 C CNN
+	1    1250 10350
+	1    0    0    -1
+$EndComp
 $EndSCHEMATC

Commit message: working on input layout
Parts:
- C101: value 100uF -> 1000uF
Changed lines of the file:
@@
 $EndDescr
 $Comp
-L GND #PWR108
+L GND #PWR01
 U 1 1 5311570D
 P 8150 7450
-F 0 "#PWR108" H 8150 7450 30  0001 C CNN
+F 0 "#PWR01" H 8150 7450 30  0001 C CNN
 F 1 "GND" H 8150 7380 30  0001 C CNN
 F 2 "" H 8150 7450 60  0000 C CNN
@@
 $EndComp
 $Comp
-L GND #PWR109
+L GND #PWR02
 U 1 1 5311577C
 P 9300 4800
-F 0 "#PWR109" H 9300 4800 30  0001 C CNN
+F 0 "#PWR02" H 9300 4800 30  0001 C CNN
 F 1 "GND" H 9300 4730 30  0001 C CNN
 F 2 "" H 9300 4800 60  0000 C CNN
@@
 $EndComp
 $Comp
-L GND #PWR103
+L GND #PWR03
 U 1 1 531157E6
 P 5050 4800
-F 0 "#PWR103" H 5050 4800 30  0001 C CNN
+F 0 "#PWR03" H 5050 4800 30  0001 C CNN
 F 1 "GND" H 5050 4730 30  0001 C CNN
 F 2 "" H 5050 4800 60  0000 C CNN
@@
 $EndComp
 $Comp
-L GND #PWR110
+L GND #PWR04
 U 1 1 53116107
 P 10650 5750
-F 0 "#PWR110" H 10650 5750 30  0001 C CNN
+F 0 "#PWR04" H 10650 5750 30  0001 C CNN
 F 1 "GND" H 10650 5680 30  0001 C CNN
 F 2 "" H 10650 5750 60  0000 C CNN
@@
 $EndComp
 $Comp
-L GND #PWR111
+L GND #PWR05
 U 1 1 53116125
 P 10950 5750
-F 0 "#PWR111" H 10950 5750 30  0001 C CNN
+F 0 "#PWR05" H 10950 5750 30  0001 C CNN
 F 1 "GND" H 10950 5680 30  0001 C CNN
 F 2 "" H 10950 5750 60  0000 C CNN
@@
 Connection ~ 11250 4200
 $Comp
-L GND #PWR112
+L GND #PWR06
 U 1 1 531163B7
 P 11250 4800
-F 0 "#PWR112" H 11250 4800 30  0001 C CNN
+F 0 "#PWR06" H 11250 4800 30  0001 C CNN
 F 1 "GND" H 11250 4730 30  0001 C CNN
 F 2 "" H 11250 4800 60  0000 C CNN
@@
 $EndComp
 $Comp
-L GND #PWR115
+L GND #PWR07
 U 1 1 53116825
 P 13050 5950
-F 0 "#PWR115" H 13050 5950 30  0001 C CNN
+F 0 "#PWR07" H 13050 5950 30  0001 C CNN
 F 1 "GND" H 13050 5880 30  0001 C CNN
 F 2 "" H 13050 5950 60  0000 C CNN
@@
 Vout\n(1.25V - 20.2V DC)
 $Comp
-L GND #PWR101
+L GND #PWR08
 U 1 1 53116888
 P 3350 4500
-F 0 "#PWR101" H 3350 4500 30  0001 C CNN
+F 0 "#PWR08" H 3350 4500 30  0001 C CNN
 F 1 "GND" H 3350 4430 30  0001 C CNN
 F 2 "" H 3350 4500 60  0000 C CNN
@@
 Connection ~ 8350 4200
 $Comp
-L GND #PWR105
+L GND #PWR09
 U 1 1 53255562
 P 5850 4800
-F 0 "#PWR105" H 5850 4800 30  0001 C CNN
+F 0 "#PWR09" H 5850 4800 30  0001 C CNN
 F 1 "GND" H 5850 4730 30  0001 C CNN
 F 2 "" H 5850 4800 60  0000 C CNN
@@
 330 & 4.7k = 19V max
 $Comp
-L GND #PWR106
+L GND #PWR010
 U 1 1 53264209
 P 6300 6700
-F 0 "#PWR106" H 6300 6700 30  0001 C CNN
+F 0 "#PWR010" H 6300 6700 30  0001 C CNN
 F 1 "GND" H 6300 6630 30  0001 C CNN
 F 2 "" H 6300 6700 60  0000 C CNN
@@
 $EndComp
 $Comp
-L GND #PWR107
+L GND #PWR011
 U 1 1 532642AB
 P 6800 6900
-F 0 "#PWR107" H 6800 6900 30  0001 C CNN
+F 0 "#PWR011" H 6800 6900 30  0001 C CNN
 F 1 "GND" H 6800 6830 30  0001 C CNN
 F 2 "" H 6800 6900 60  0000 C CNN
@@
 	5350 6300 6000 6300
 $Comp
-L GND #PWR104
+L GND #PWR012
 U 1 1 5326496C
 P 5800 6900
-F 0 "#PWR104" H 5800 6900 30  0001 C CNN
+F 0 "#PWR012" H 5800 6900 30  0001 C CNN
 F 1 "GND" H 5800 6830 30  0001 C CNN
 F 2 "" H 5800 6900 60  0000 C CNN
@@
 5V
 $Comp
-L GND #PWR114
+L GND #PWR013
 U 1 1 53267BC5
 P 11950 5550
-F 0 "#PWR114" H 11950 5550 30  0001 C CNN
+F 0 "#PWR013" H 11950 5550 30  0001 C CNN
 F 1 "GND" H 11950 5480 30  0001 C CNN
 F 2 "" H 11950 5550 60  0000 C CNN
@@
 P 5050 4500
 F 0 "C101" H 5070 4560 30  0000 L BNN
-F 1 "100uF" H 5070 4410 30  0000 L TNN
+F 1 "1000uF" H 5070 4410 30  0000 L TNN
 F 2 "~" H 5088 4350 30  0000 C CNN
 F 3 "~" H 5050 4500 60  0000 C CNN
@@
 $EndComp
 $Comp
-L GND #PWR113
+L GND #PWR014
 U 1 1 532B868B
 P 11850 3200
-F 0 "#PWR113" H 11850 3200 30  0001 C CNN
+F 0 "#PWR014" H 11850 3200 30  0001 C CNN
 F 1 "GND" H 11850 3130 30  0001 C CNN
 F 2 "" H 11850 3200 60  0000 C CNN
@@
 $EndComp
 $Comp
-L GND #PWR102
+L GND #PWR015
 U 1 1 532F0044
 P 3350 5100
-F 0 "#PWR102" H 3350 5100 30  0001 C CNN
+F 0 "#PWR015" H 3350 5100 30  0001 C CNN
 F 1 "GND" H 3350 5030 30  0001 C CNN
 F 2 "" H 3350 5100 60  0000 C CNN

Commit message: working on layout
Connections:
- wire segments 85 -> 89
Changed lines of the file:
@@
 F0 "current_limit_r" 50
 F1 "current_limit_r.sch" 50
-F2 "IN" I L 7350 4200 60
-F3 "OUT" O R 8200 4200 60
+F2 "R_LIM+" I L 7350 4100 60
+F3 "R_LIM-" O R 8200 4300 60
 $EndSheet
-Wire Wire Line
-	7000 4200 7350 4200
 Connection ~ 7200 4200
 Wire Wire Line
@@
 Wire Wire Line
 	6050 3500 6750 3500
-Wire Wire Line
-	8200 4200 9650 4200
 Wire Notes Line
 	5600 2800 8600 2800
@@
 	1    0    0    -1
 $EndComp
+Wire Wire Line
+	7000 4200 7300 4200
+Wire Wire Line
+	7300 4200 7300 4100
+Wire Wire Line
+	7300 4100 7350 4100
+Wire Wire Line
+	8250 4200 9650 4200
+Wire Wire Line
+	8250 4200 8250 4300
+Wire Wire Line
+	8250 4300 8200 4300
 $EndSCHEMATC

Commit message: pulling in diodes lib
Parts:
- P101: value CONN_1 -> Vout+
- P102: value CONN_1 -> Vout-
Changed lines of the file:
@@
 P 13300 4200
 F 0 "P101" H 13380 4200 40  0000 L CNN
-F 1 "CONN_1" H 13300 4255 30  0001 C CNN
+F 1 "Vout+" H 13300 4255 30  0001 C CNN
 F 2 "" H 13300 4200 60  0000 C CNN
 F 3 "" H 13300 4200 60  0000 C CNN
@@
 P 13300 4600
 F 0 "P102" H 13380 4600 40  0000 L CNN
-F 1 "CONN_1" H 13300 4655 30  0001 C CNN
+F 1 "Vout-" H 13300 4655 30  0001 C CNN
 F 2 "" H 13300 4600 60  0000 C CNN
 F 3 "" H 13300 4600 60  0000 C CNN

Commit message: adding voltmeter and potentiometer to layout
Parts:
- removed RV101: 4k7, ~, symbol POT
- added RV101: 4.7k, ~, symbol POT_10T
Changed lines of the file:
@@
-$EndComp
-$Comp
-L POT RV101
-U 1 1 531160F8
-P 10650 5400
-F 0 "RV101" H 10650 5300 50  0000 C CNN
-F 1 "4k7" H 10650 5400 50  0000 C CNN
-F 2 "~" H 10650 5400 60  0000 C CNN
-F 3 "~" H 10650 5400 60  0000 C CNN
-	1    10650 5400
-	0    -1   -1   0
 $EndComp
 $Comp
@@
 Text Notes 5600 5925 0    60   ~ 0
 5V Supply
-$Comp
-L VOLTMETER DS101
-U 1 1 53267314
-P 12050 3000
-F 0 "DS101" H 12100 3150 40  0000 L CNN
-F 1 "VOLTMETER" H 12900 2600 40  0000 R CNN
-F 2 "~" H 12880 3400 60  0000 C CNN
-F 3 "~" H 12880 3400 60  0000 C CNN
-	1    12050 3000
-	1    0    0    -1
-$EndComp
 Text GLabel 11850 2900 1    40   Input ~ 0
 5V
@@
 Wire Wire Line
 	8250 4300 8200 4300
+$Comp
+L POT_10T RV101
+U 1 1 532F65CA
+P 10650 5400
+F 0 "RV101" H 10475 5485 30  0000 C CNN
+F 1 "4.7k" H 10845 5360 30  0000 C CNN
+F 2 "~" H 10650 5400 60  0000 C CNN
+F 3 "~" H 10650 5400 60  0000 C CNN
+	1    10650 5400
+	0    -1   -1   0
+$EndComp
+$Comp
+L VOLTMETER DS101
+U 1 1 532F70BB
+P 12050 3000
+F 0 "DS101" H 12100 3150 40  0000 L CNN
+F 1 "VOLTMETER" H 12900 2600 40  0000 R CNN
+F 2 "~" H 12880 3400 60  0000 C CNN
+F 3 "~" H 12880 3400 60  0000 C CNN
+	1    12050 3000
+	1    0    0    -1
+$EndComp
 $EndSCHEMATC
