File: DualLM317BenchSupply/$DualLM317BenchSupply.sch (KiCad schematic (older format))
At the start: 31 parts, among them CON101 BARREL_JACK, CON102 BARREL_JACK, P101 Vout+, P102 Vout-, SW101 SPDT, SW102 SPDT, SW103 SPDT, U101 78L05, U102 LM317, U103 LM317

Commit message: correcting pads for ammeter and running traces to it
Parts:
- gave numbers to parts that had none: 1
Changed lines of the file:
@@
 $EndComp
 $Comp
-L AMMETER_V DS?
+L AMMETER_V DS102
 U 1 1 5334CAF5
 P 12050 5350
-F 0 "DS?" H 12100 5500 40  0000 L CNN
+F 0 "DS102" H 12100 5500 40  0000 L CNN
 F 1 "AMMETER_V" H 12900 4950 40  0000 R CNN
 F 2 "~" H 12880 5750 60  0000 C CNN
